File: electrical/control board/_saved_control board.sch (KiCad schematic (older format))
At the start: 68 parts, among them J1 analog_extra, J10 Motor_2, J11 Motor_3, J12 Motor_4, J13 Motor_5, J14 Motor_6, J15 Motor_7, J16 Motor_8, J2 Programming_Header, J3 Conn_01x08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

Commit message: Finally got the correct board outline in Kicad
Parts:
- gave numbers to parts that had none: 1
Connections:
- wire segments 322 -> 328
Changed lines of the file:
@@
 Wire Wire Line
 	4650 1650 4450 1650
-Wire Wire Line
-	4650 1300 4450 1300
-Wire Wire Line
-	4650 900  4400 900
 $Comp
 L power:GND #PWR0144
@@
 Consider moving to power board
 $Comp
-L Connector_Generic:Conn_02x04_Counter_Clockwise J?
+L Connector_Generic:Conn_02x04_Counter_Clockwise J7
 U 1 1 5C362818
 P 8800 5600
-F 0 "J?" H 8850 5917 50  0000 C CNN
+F 0 "J7" H 8850 5917 50  0000 C CNN
 F 1 "Power_Connector" H 8850 5826 50  0000 C CNN
 F 2 "" H 8800 5600 50  0001 C CNN
@@
 $EndComp
 $Comp
-L power:+3.3V #PWR?
+L power:+3.3V #PWR0101
 U 1 1 5C362D91
 P 9700 5750
-F 0 "#PWR?" H 9700 5600 50  0001 C CNN
+F 0 "#PWR0101" H 9700 5600 50  0001 C CNN
 F 1 "+3.3V" H 9715 5923 50  0000 C CNN
 F 2 "" H 9700 5750 50  0001 C CNN
@@
 $EndComp
 $Comp
-L power:+5V #PWR?
+L power:+5V #PWR0117
 U 1 1 5C362F15
 P 9500 5650
-F 0 "#PWR?" H 9500 5500 50  0001 C CNN
+F 0 "#PWR0117" H 9500 5500 50  0001 C CNN
 F 1 "+5V" H 9515 5823 50  0000 C CNN
 F 2 "" H 9500 5650 50  0001 C CNN
@@
 $EndComp
 $Comp
-L power:+24V #PWR?
+L power:+24V #PWR0118
 U 1 1 5C3952B5
 P 9350 5550
-F 0 "#PWR?" H 9350 5400 50  0001 C CNN
+F 0 "#PWR0118" H 9350 5400 50  0001 C CNN
 F 1 "+24V" H 9365 5723 50  0000 C CNN
 F 2 "" H 9350 5550 50  0001 C CNN
@@
 $EndComp
 $Comp
-L power:+48V #PWR?
+L power:+48V #PWR0119
 U 1 1 5C395374
 P 9200 5450
-F 0 "#PWR?" H 9200 5300 50  0001 C CNN
+F 0 "#PWR0119" H 9200 5300 50  0001 C CNN
 F 1 "+48V" H 9215 5623 50  0000 C CNN
 F 2 "" H 9200 5450 50  0001 C CNN
@@
 	9200 5500 9200 5450
 $Comp
-L power:GND #PWR?
+L power:GND #PWR0120
 U 1 1 5C47CCF8
 P 8450 5850
-F 0 "#PWR?" H 8450 5600 50  0001 C CNN
+F 0 "#PWR0120" H 8450 5600 50  0001 C CNN
 F 1 "GND" H 8455 5677 50  0000 C CNN
 F 2 "" H 8450 5850 50  0001 C CNN
@@
 Wire Wire Line
 	8450 5800 8450 5850
+Wire Wire Line
+	4450 1650 4450 2400
+Wire Wire Line
+	4450 2400 3750 2400
+Wire Wire Line
+	4400 2300 3750 2300
+Wire Wire Line
+	4400 1300 4650 1300
+Wire Wire Line
+	4400 1300 4400 2300
+Wire Wire Line
+	4350 900  4350 2200
+Wire Wire Line
+	4350 2200 3750 2200
+Wire Wire Line
+	4350 900  4650 900
 $EndSCHEMATC
