File: electrical/control board/control board.sch (KiCad schematic (older format))
At the start: 68 parts, among them J1 analog_extra, J10 Motor_2, J11 Motor_3, J12 Motor_4, J13 Motor_5, J14 Motor_6, J15 Motor_7, J16 Motor_8, J2 Programming_Header, J3 Conn_01x08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

Commit message: Moved current measurement to power board
Parts:
- removed C11: C_Small, Capacitor_SMD:C_0603_1608Metric_Pad1.05x0.95mm_HandSolder, symbol Device:C_Small
- removed R6: 1m, footprints:FC4L64, symbol Device:R_Shunt
- removed U3: INA240-INA240, Package_SO:TSSOP-8_4.4x3mm_P0.65mm, symbol custom_symbols:INA240-INA240
Connections:
- net labels removed: 48V_IN
- wire segments 328 -> 313
Other:
- note added: "Add header space for current measurement"
Changed lines of the file:
@@
 Voltage Monitering
-$Comp
-L Device:R_Shunt R6
-U 1 1 5C076A09
-P 3800 5850
-F 0 "R6" H 3712 5896 50  0000 R CNN
-F 1 "1m" H 3712 5805 50  0000 R CNN
-F 2 "footprints:FC4L64" V 3730 5850 50  0001 C CNN
-F 3 "~" H 3800 5850 50  0001 C CNN
-	1    3800 5850
-	1    0    0    -1
-$EndComp
-$Comp
-L custom_symbols:INA240-INA240 U3
-U 1 1 5C085EBE
-P 4400 5850
-F 0 "U3" H 4400 6225 50  0000 C CNN
-F 1 "INA240-INA240" H 4400 6134 50  0000 C CNN
-F 2 "Package_SO:TSSOP-8_4.4x3mm_P0.65mm" H 4400 5850 50  0001 C CNN
-F 3 "" H 4400 5850 50  0001 C CNN
-	1    4400 5850
-	1    0    0    -1
-$EndComp
-Wire Wire Line
-	4050 5800 3950 5800
-Wire Wire Line
-	3950 5800 3950 5750
-Wire Wire Line
-	4050 5900 3950 5900
-Wire Wire Line
-	3950 5900 3950 5950
 $Comp
 L Device:LED D1
@@
 	7100 9550 7100 9500
 $Comp
-L power:+48V #PWR0151
-U 1 1 5BFA8577
-P 3400 6050
-F 0 "#PWR0151" H 3400 5900 50  0001 C CNN
-F 1 "+48V" H 3415 6223 50  0000 C CNN
-F 2 "" H 3400 6050 50  0001 C CNN
-F 3 "" H 3400 6050 50  0001 C CNN
-	1    3400 6050
-	1    0    0    -1
-$EndComp
-Wire Wire Line
-	3800 6050 3400 6050
-Text Label 3800 5550 0    50   ~ 0
-48V_IN
-Wire Wire Line
-	3800 5650 3800 5550
-$Comp
-L power:GND #PWR0152
-U 1 1 5BFE347A
-P 4950 6200
-F 0 "#PWR0152" H 4950 5950 50  0001 C CNN
-F 1 "GND" H 4955 6027 50  0000 C CNN
-F 2 "" H 4950 6200 50  0001 C CNN
-F 3 "" H 4950 6200 50  0001 C CNN
-	1    4950 6200
-	1    0    0    -1
-$EndComp
-Wire Wire Line
-	4750 5800 4950 5800
-Wire Wire Line
-	4950 5800 4950 5900
-Wire Wire Line
-	4750 5900 4950 5900
-Connection ~ 4950 5900
-$Comp
 L Device:LED D4
 U 1 1 5C00BD15
@@
 	4850 2350 4850 2750
 Connection ~ 4850 2750
-$Comp
-L power:GND #PWR0154
-U 1 1 5C0DE6A1
-P 4000 6100
-F 0 "#PWR0154" H 4000 5850 50  0001 C CNN
-F 1 "GND" H 4005 5927 50  0000 C CNN
-F 2 "" H 4000 6100 50  0001 C CNN
-F 3 "" H 4000 6100 50  0001 C CNN
-	1    4000 6100
-	1    0    0    -1
-$EndComp
-Wire Wire Line
-	4050 6000 4000 6000
-Wire Wire Line
-	4000 6000 4000 6100
-$Comp
-L Device:C_Small C11
-U 1 1 5C10BBA8
-P 5050 6100
-F 0 "C11" H 5142 6146 50  0000 L CNN
-F 1 "C_Small" H 5142 6055 50  0000 L CNN
-F 2 "Capacitor_SMD:C_0603_1608Metric_Pad1.05x0.95mm_HandSolder" H 5050 6100 50  0001 C CNN
-F 3 "~" H 5050 6100 50  0001 C CNN
-	1    5050 6100
-	1    0    0    -1
-$EndComp
-Wire Wire Line
-	4950 5900 4950 6200
-Wire Wire Line
-	5050 6200 4950 6200
-Connection ~ 4950 6200
-Wire Wire Line
-	4750 6000 5050 6000
-$Comp
-L power:+3.3V #PWR0155
-U 1 1 5C167660
-P 5050 5900
-F 0 "#PWR0155" H 5050 5750 50  0001 C CNN
-F 1 "+3.3V" H 5065 6073 50  0000 C CNN
-F 2 "" H 5050 5900 50  0001 C CNN
-F 3 "" H 5050 5900 50  0001 C CNN
-	1    5050 5900
-	1    0    0    -1
-$EndComp
-Wire Wire Line
-	5050 5900 5050 6000
-Connection ~ 5050 6000
 Text Label 1600 3900 0    50   ~ 0
 CURRENT_MEASURE
 Wire Wire Line
 	1600 3900 2350 3900
-Text Label 4750 5700 0    50   ~ 0
-CURRENT_MEASURE
 $Comp
 L Transistor_BJT:DTC114E Q2
@@
 Wire Wire Line
 	4350 900  4650 900
+Text Notes 6800 6900 0    50   ~ 0
+Add header space for current measurement
 $EndSCHEMATC

Commit message: routed voltage measurement
Other:
- note added: "This ICM won't work. Find a new one that can be soldered"
Changed lines of the file:
@@
 Text Notes 6800 6900 0    50   ~ 0
 Add header space for current measurement
+Text Notes 9600 7650 0    50   ~ 0
+This ICM won't work. Find a new one that can be soldered
 $EndSCHEMATC

Commit message: found a crystal
Parts:
- Y1: footprint (none) -> Crystal:Crystal_HC49-U_Vertical; digikey # (none) -> CTX917-ND‎
Changed lines of the file:
@@
 F 0 "Y1" V 1854 3281 50  0000 L CNN
 F 1 "8Mhz" V 1945 3281 50  0000 L CNN
-F 2 "" H 1900 3150 50  0001 C CNN
+F 2 "Crystal:Crystal_HC49-U_Vertical" H 1900 3150 50  0001 C CNN
 F 3 "~" H 1900 3150 50  0001 C CNN
+F 4 "CTX917-ND‎" V 1900 3150 50  0001 C CNN "digikey #"
 	1    1900 3150
 	0    1    1    0

Commit message: Found parts for LEDs
Parts:
- D1, D4: value LED -> LED-RED; Digikey part number (none) -> SML-D12U1WT86CT-ND
- D2, D5: value LED -> LED-YELLOW; Digikey part number (none) -> 160-1448-1-ND
- D3, D6: value LED -> LED-GREEN; Digikey part number (none) -> 160-1446-1-ND
- J7: Digikey # WM3803-ND -> (none); Digikey part number (none) -> WM3803-ND
- Y1: Digikey part number (none) -> CTX917-ND‎; digikey # CTX917-ND‎ -> (none)
Changed lines of the file:
@@
 F 2 "Crystal:Crystal_HC49-U_Vertical" H 1900 3150 50  0001 C CNN
 F 3 "~" H 1900 3150 50  0001 C CNN
-F 4 "CTX917-ND‎" V 1900 3150 50  0001 C CNN "digikey #"
+F 4 "" V 1900 3150 50  0001 C CNN "digikey #"
+F 5 "CTX917-ND‎" H 0   0   50  0001 C CNN "Digikey part number"
 	1    1900 3150
 	0    1    1    0
@@
 P 5150 900
 F 0 "D1" H 5142 645 50  0000 C CNN
-F 1 "LED" H 5142 736 50  0000 C CNN
+F 1 "LED-RED" H 5142 736 50  0000 C CNN
 F 2 "" H 5150 900 50  0001 C CNN
-F 3 "~" H 5150 900 50  0001 C CNN
+F 3 "https://www.rohm.com/datasheet/SML-D12U1W" H 5150 900 50  0001 C CNN
+F 4 "SML-D12U1WT86CT-ND " H 0   0   50  0001 C CNN "Digikey part number"
 	1    5150 900
 	-1   0    0    1
@@
 P 5150 1650
 F 0 "D3" H 5142 1395 50  0000 C CNN
-F 1 "LED" H 5142 1486 50  0000 C CNN
+F 1 "LED-GREEN" H 5142 1486 50  0000 C CNN
 F 2 "" H 5150 1650 50  0001 C CNN
-F 3 "~" H 5150 1650 50  0001 C CNN
+F 3 "http://optoelectronics.liteon.com/upload/download/DS22-2000-228/LTST-C191KGKT.PDF" H 5150 1650 50  0001 C CNN
+F 4 "160-1446-1-ND " H 0   0   50  0001 C CNN "Digikey part number"
 	1    5150 1650
 	-1   0    0    1
@@
 P 5150 1300
 F 0 "D2" H 5142 1045 50  0000 C CNN
-F 1 "LED" H 5142 1136 50  0000 C CNN
+F 1 "LED-YELLOW" H 5142 1136 50  0000 C CNN
 F 2 "" H 5150 1300 50  0001 C CNN
-F 3 "~" H 5150 1300 50  0001 C CNN
+F 3 "http://optoelectronics.liteon.com/upload/download/DS22-2000-224/LTST-C191KSKT.PDF" H 5150 1300 50  0001 C CNN
+F 4 "160-1448-1-ND " H 0   0   50  0001 C CNN "Digikey part number"
 	1    5150 1300
 	-1   0    0    1
@@
 P 5200 2350
 F 0 "D4" H 5191 2566 50  0000 C CNN
-F 1 "LED" H 5191 2475 50  0000 C CNN
+F 1 "LED-RED" H 5191 2475 50  0000 C CNN
 F 2 "" H 5200 2350 50  0001 C CNN
-F 3 "~" H 5200 2350 50  0001 C CNN
+F 3 "https://www.rohm.com/datasheet/SML-D12U1W" H 5200 2350 50  0001 C CNN
+F 4 "SML-D12U1WT86CT-ND " H 0   0   50  0001 C CNN "Digikey part number"
 	1    5200 2350
 	1    0    0    -1
@@
 P 5200 3100
 F 0 "D6" H 5191 3316 50  0000 C CNN
-F 1 "LED" H 5191 3225 50  0000 C CNN
+F 1 "LED-GREEN" H 5191 3225 50  0000 C CNN
 F 2 "" H 5200 3100 50  0001 C CNN
-F 3 "~" H 5200 3100 50  0001 C CNN
+F 3 "http://optoelectronics.liteon.com/upload/download/DS22-2000-228/LTST-C191KGKT.PDF" H 5200 3100 50  0001 C CNN
+F 4 "160-1446-1-ND " H 0   0   50  0001 C CNN "Digikey part number"
 	1    5200 3100
 	1    0    0    -1
@@
 P 5200 2750
 F 0 "D5" H 5191 2966 50  0000 C CNN
-F 1 "LED" H 5191 2875 50  0000 C CNN
+F 1 "LED-YELLOW" H 5191 2875 50  0000 C CNN
 F 2 "" H 5200 2750 50  0001 C CNN
-F 3 "~" H 5200 2750 50  0001 C CNN
+F 3 "http://optoelectronics.liteon.com/upload/download/DS22-2000-224/LTST-C191KSKT.PDF" H 5200 2750 50  0001 C CNN
+F 4 "160-1448-1-ND " H 0   0   50  0001 C CNN "Digikey part number"
 	1    5200 2750
 	1    0    0    -1
@@
 F 2 "Connector_Molex:Molex_Mini-Fit_Jr_5566-08A2_2x04_P4.20mm_Vertical" H 8800 5600 50  0001 C CNN
 F 3 "~" H 8800 5600 50  0001 C CNN
-F 4 "WM3803-ND " H 8800 5600 50  0001 C CNN "Digikey #"
+F 4 "" H 8800 5600 50  0001 C CNN "Digikey #"
+F 5 "WM3803-ND " H 0   0   50  0001 C CNN "Digikey part number"
 	1    8800 5600
 	1    0    0    -1

Commit message: created hand solder footprint for microcontoller
Parts:
- D1, D2, D3, D4, D5, D6: footprint (none) -> LED_SMD:LED_0603_1608Metric_Pad1.05x0.95mm_HandSolder
- U1: footprint Package_QFP:LQFP-64_10x10mm_P0.5mm -> footprints:LQFP-64_10x10mm_P0.5mm_handsolder
Changed lines of the file:
@@
 F 0 "U1" H 3050 1614 50  0000 C CNN
 F 1 "STM32F446RETx" H 3050 1523 50  0000 C CNN
-F 2 "Package_QFP:LQFP-64_10x10mm_P0.5mm" H 2450 1800 50  0001 R CNN
+F 2 "footprints:LQFP-64_10x10mm_P0.5mm_handsolder" H 2450 1800 50  0001 R CNN
 F 3 "http://www.st.com/st-web-ui/static/active/en/resource/technical/document/datasheet/DM00141306.pdf" H 3050 3500 50  0001 C CNN
 	1    3050 3500
@@
 F 0 "D1" H 5142 645 50  0000 C CNN
 F 1 "LED-RED" H 5142 736 50  0000 C CNN
-F 2 "" H 5150 900 50  0001 C CNN
+F 2 "LED_SMD:LED_0603_1608Metric_Pad1.05x0.95mm_HandSolder" H 5150 900 50  0001 C CNN
 F 3 "https://www.rohm.com/datasheet/SML-D12U1W" H 5150 900 50  0001 C CNN
 F 4 "SML-D12U1WT86CT-ND " H 0   0   50  0001 C CNN "Digikey part number"
@@
 F 0 "D3" H 5142 1395 50  0000 C CNN
 F 1 "LED-GREEN" H 5142 1486 50  0000 C CNN
-F 2 "" H 5150 1650 50  0001 C CNN
+F 2 "LED_SMD:LED_0603_1608Metric_Pad1.05x0.95mm_HandSolder" H 5150 1650 50  0001 C CNN
 F 3 "http://optoelectronics.liteon.com/upload/download/DS22-2000-228/LTST-C191KGKT.PDF" H 5150 1650 50  0001 C CNN
 F 4 "160-1446-1-ND " H 0   0   50  0001 C CNN "Digikey part number"
@@
 F 0 "D2" H 5142 1045 50  0000 C CNN
 F 1 "LED-YELLOW" H 5142 1136 50  0000 C CNN
-F 2 "" H 5150 1300 50  0001 C CNN
+F 2 "LED_SMD:LED_0603_1608Metric_Pad1.05x0.95mm_HandSolder" H 5150 1300 50  0001 C CNN
 F 3 "http://optoelectronics.liteon.com/upload/download/DS22-2000-224/LTST-C191KSKT.PDF" H 5150 1300 50  0001 C CNN
 F 4 "160-1448-1-ND " H 0   0   50  0001 C CNN "Digikey part number"
@@
 F 0 "D4" H 5191 2566 50  0000 C CNN
 F 1 "LED-RED" H 5191 2475 50  0000 C CNN
-F 2 "" H 5200 2350 50  0001 C CNN
+F 2 "LED_SMD:LED_0603_1608Metric_Pad1.05x0.95mm_HandSolder" H 5200 2350 50  0001 C CNN
 F 3 "https://www.rohm.com/datasheet/SML-D12U1W" H 5200 2350 50  0001 C CNN
 F 4 "SML-D12U1WT86CT-ND " H 0   0   50  0001 C CNN "Digikey part number"
@@
 F 0 "D6" H 5191 3316 50  0000 C CNN
 F 1 "LED-GREEN" H 5191 3225 50  0000 C CNN
-F 2 "" H 5200 3100 50  0001 C CNN
+F 2 "LED_SMD:LED_0603_1608Metric_Pad1.05x0.95mm_HandSolder" H 5200 3100 50  0001 C CNN
 F 3 "http://optoelectronics.liteon.com/upload/download/DS22-2000-228/LTST-C191KGKT.PDF" H 5200 3100 50  0001 C CNN
 F 4 "160-1446-1-ND " H 0   0   50  0001 C CNN "Digikey part number"
@@
 F 0 "D5" H 5191 2966 50  0000 C CNN
 F 1 "LED-YELLOW" H 5191 2875 50  0000 C CNN
-F 2 "" H 5200 2750 50  0001 C CNN
+F 2 "LED_SMD:LED_0603_1608Metric_Pad1.05x0.95mm_HandSolder" H 5200 2750 50  0001 C CNN
 F 3 "http://optoelectronics.liteon.com/upload/download/DS22-2000-224/LTST-C191KSKT.PDF" H 5200 2750 50  0001 C CNN
 F 4 "160-1448-1-ND " H 0   0   50  0001 C CNN "Digikey part number"

Commit message: Changed pins on motors
Connections:
- net labels added: MOTOR_1, MOTOR_2, MOTOR_3, MOTOR_4, MOTOR_5, MOTOR_6, MOTOR_7, MOTOR_8
- wire segments 313 -> 296
Changed lines of the file:
@@
 Text Label 2000 4700 0    50   ~ 0
 MISC_RX
-Text Label 1800 4800 0    50   ~ 0
+Text Label 1800 5200 0    50   ~ 0
 UART5_TX
 Text Label 1850 4100 0    50   ~ 0
@@
 Text Label 3750 3800 0    50   ~ 0
 SWITCH_B
-Text Label 3750 3900 0    50   ~ 0
-SWITCH_C
+Text Label 2000 3400 0    50   ~ 0
+MOTOR_6
 Text Label 3750 4100 0    50   ~ 0
-SWITCH_D
+MOTOR_5
 Wire Wire Line
 	4800 9000 4800 8700
@@
 	-1   0    0    1
 $EndComp
-Wire Wire Line
-	3900 3450 3900 3500
-Wire Wire Line
-	3900 3500 3750 3500
-Wire Wire Line
-	3900 3450 7000 3450
-Wire Wire Line
-	7000 3800 4300 3800
-Wire Wire Line
-	4300 3800 4300 4500
-Wire Wire Line
-	4300 4500 3750 4500
-Wire Wire Line
-	7000 4150 4400 4150
-Wire Wire Line
-	4400 4150 4400 4600
-Wire Wire Line
-	4400 4600 3750 4600
-Wire Wire Line
-	7000 4500 4550 4500
-Wire Wire Line
-	4550 4500 4550 4700
-Wire Wire Line
-	4550 4700 3750 4700
-Wire Wire Line
-	7000 4850 4550 4850
-Wire Wire Line
-	4550 4850 4550 4800
-Wire Wire Line
-	4550 4800 3750 4800
-Wire Wire Line
-	7000 5200 4450 5200
-Wire Wire Line
-	4450 5200 4450 4900
-Wire Wire Line
-	4450 4900 3750 4900
-Wire Wire Line
-	7000 5550 6700 5550
-Wire Wire Line
-	6700 5550 6700 5250
-Wire Wire Line
-	6700 5250 4350 5250
-Wire Wire Line
-	4350 5250 4350 5000
-Wire Wire Line
-	3750 5000 4350 5000
-Wire Wire Line
-	3750 5100 4250 5100
-Wire Wire Line
-	4250 5100 4250 5300
-Wire Wire Line
-	4250 5300 6650 5300
-Wire Wire Line
-	6650 5300 6650 5900
-Wire Wire Line
-	6650 5900 7000 5900
 $Comp
 L power:GND #PWR0125
@@
 Text Notes 9600 7650 0    50   ~ 0
 This ICM won't work. Find a new one that can be soldered
+Text Label 6650 3450 0    50   ~ 0
+MOTOR_1
+Text Label 6650 3800 0    50   ~ 0
+MOTOR_2
+Text Label 6650 4150 0    50   ~ 0
+MOTOR_3
+Text Label 6650 4500 0    50   ~ 0
+MOTOR_4
+Text Label 6650 4850 0    50   ~ 0
+MOTOR_5
+Text Label 6650 5200 0    50   ~ 0
+MOTOR_6
+Text Label 6650 5550 0    50   ~ 0
+MOTOR_7
+Text Label 6650 5900 0    50   ~ 0
+MOTOR_8
+Wire Wire Line
+	7000 5900 6650 5900
+Wire Wire Line
+	7000 5550 6650 5550
+Wire Wire Line
+	7000 5200 6650 5200
+Wire Wire Line
+	7000 4850 6650 4850
+Wire Wire Line
+	7000 4500 6650 4500
+Wire Wire Line
+	7000 4150 6650 4150
+Wire Wire Line
+	7000 3800 6650 3800
+Wire Wire Line
+	7000 3450 6650 3450
+Text Label 3750 4600 0    50   ~ 0
+MOTOR_2
+Text Label 3750 4500 0    50   ~ 0
+MOTOR_3
+Text Label 3750 4200 0    50   ~ 0
+MOTOR_4
+Text Label 2000 4800 0    50   ~ 0
+MOTOR_7
+Wire Wire Line
+	2000 4800 2350 4800
+Text Label 3750 3500 0    50   ~ 0
+MOTOR_8
+Text Label 2000 5100 0    50   ~ 0
+MOTOR_1
+Wire Wire Line
+	2350 5100 2000 5100
+Wire Wire Line
+	2000 3400 2350 3400
 $EndSCHEMATC

Commit message: found parts for most of the stuff on the control board
Parts:
- removed J3: Conn_01x08, Connector_PinHeader_2.54mm:PinHeader_1x08_P2.54mm_Vertical, symbol Connector_Generic:Conn_01x08
- removed Q1, Q3, Q4, Q5: Q_NMOS_GDS, symbol Device:Q_NMOS_GDS
- removed R12, R3, R4, R5: 10k, Resistor_SMD:R_0603_1608Metric_Pad1.05x0.95mm_HandSolder, symbol Device:R_Small
- C1, C10, C5, C6, C7, C8, C9: Digikey part number (none) -> 1276-1005-1-ND
- C13, C14, C4: Digikey part number (none) -> 1276-1102-1-ND
- C15, C17, C18: value .1uF -> 0.1uF; Digikey part number (none) -> 1276-1005-1-ND
- C2, C3: Digikey part number (none) -> 1276-1021-1-ND
- P1: Digikey part number (none) -> n/a
- Q2: Digikey part number (none) -> DTC114EET1GOSCT-ND
- R1, R2: Digikey part number (none) -> CR0603-JW-472ELFCT-ND
- R13, R7: Digikey part number (none) -> CR0603-JW-103ELFCT-ND
- R14: Digikey part number (none) -> CR0603-JW-123ELFCT-ND
- R15: Digikey part number (none) -> CR0603-JW-104ELFCT-ND
- R16: Digikey part number (none) -> RMCF0603JT3K60CT-ND
- R8: Digikey part number (none) -> RMCF0603JT56K0CT-ND
- U1: Digikey part number (none) -> 497-15376-ND
- U2: Digikey part number (none) -> HIH7130-000-001CT-ND
- U7: Digikey part number (none) -> 1428-1061-1-ND‎
Connections:
- net labels removed: SWITCH_C, SWITCH_D
- wire segments 296 -> 251

Commit message: replaced the motor headers
Parts:
- J10, J11, J12, J13, J14, J15, J16, J5: footprint Connector_PinHeader_2.54mm:PinHeader_1x03_P2.54mm_Vertical -> Connector_Harwin:Harwin_LTek-Male_03_P2.00mm_Vertical; Digikey part number (none) -> 952-1070-5-ND‎
- J4, J6: footprint Connector_PinHeader_2.54mm:PinHeader_1x04_P2.54mm_Vertical -> Connector_Harwin:Harwin_LTek-Male_04_P2.00mm_Vertical; Digikey part number (none) -> 952-1071-5-ND
Changed lines of the file:
@@
 F 0 "J4" H 7378 9626 50  0000 L CNN
 F 1 "datamate_sensors" H 7378 9535 50  0000 L CNN
-F 2 "Connector_PinHeader_2.54mm:PinHeader_1x04_P2.54mm_Vertical" H 7350 9650 50  0001 C CNN
+F 2 "Connector_Harwin:Harwin_LTek-Male_04_P2.00mm_Vertical" H 7350 9650 50  0001 C CNN
 F 3 "~" H 7350 9650 50  0001 C CNN
+F 4 "952-1071-5-ND" H 0   0   50  0001 C CNN "Digikey part number"
 	1    7350 9650
 	1    0    0    -1
@@
 F 0 "J6" H 7277 10626 50  0000 L CNN
 F 1 "datamate_misc" H 7277 10535 50  0000 L CNN
-F 2 "Connector_PinHeader_2.54mm:PinHeader_1x04_P2.54mm_Vertical" H 7250 10650 50  0001 C CNN
+F 2 "Connector_Harwin:Harwin_LTek-Male_04_P2.00mm_Vertical" H 7250 10650 50  0001 C CNN
 F 3 "~" H 7250 10650 50  0001 C CNN
+F 4 "952-1071-5-ND" H 0   0   50  0001 C CNN "Digikey part number"
 	1    7250 10650
 	1    0    0    -1
@@
 F 0 "J5" H 7172 3480 50  0000 R CNN
 F 1 "Motor_1" H 7172 3571 50  0000 R CNN
-F 2 "Connector_PinHeader_2.54mm:PinHeader_1x03_P2.54mm_Vertical" H 7200 3550 50  0001 C CNN
+F 2 "Connector_Harwin:Harwin_LTek-Male_03_P2.00mm_Vertical" H 7200 3550 50  0001 C CNN
 F 3 "~" H 7200 3550 50  0001 C CNN
+F 4 "952-1070-5-ND‎" H 0   0   50  0001 C CNN "Digikey part number"
 	1    7200 3550
 	-1   0    0    1
@@
 F 0 "J10" H 7172 3830 50  0000 R CNN
 F 1 "Motor_2" H 7172 3921 50  0000 R CNN
-F 2 "Connector_PinHeader_2.54mm:PinHeader_1x03_P2.54mm_Vertical" H 7200 3900 50  0001 C CNN
+F 2 "Connector_Harwin:Harwin_LTek-Male_03_P2.00mm_Vertical" H 7200 3900 50  0001 C CNN
 F 3 "~" H 7200 3900 50  0001 C CNN
+F 4 "952-1070-5-ND‎" H 0   0   50  0001 C CNN "Digikey part number"
 	1    7200 3900
 	-1   0    0    1
@@
 F 0 "J11" H 7172 4180 50  0000 R CNN
 F 1 "Motor_3" H 7172 4271 50  0000 R CNN
-F 2 "Connector_PinHeader_2.54mm:PinHeader_1x03_P2.54mm_Vertical" H 7200 4250 50  0001 C CNN
+F 2 "Connector_Harwin:Harwin_LTek-Male_03_P2.00mm_Vertical" H 7200 4250 50  0001 C CNN
 F 3 "~" H 7200 4250 50  0001 C CNN
+F 4 "952-1070-5-ND‎" H 0   0   50  0001 C CNN "Digikey part number"
 	1    7200 4250
 	-1   0    0    1
@@
 F 0 "J12" H 7172 4530 50  0000 R CNN
 F 1 "Motor_4" H 7172 4621 50  0000 R CNN
-F 2 "Connector_PinHeader_2.54mm:PinHeader_1x03_P2.54mm_Vertical" H 7200 4600 50  0001 C CNN
+F 2 "Connector_Harwin:Harwin_LTek-Male_03_P2.00mm_Vertical" H 7200 4600 50  0001 C CNN
 F 3 "~" H 7200 4600 50  0001 C CNN
+F 4 "952-1070-5-ND‎" H 0   0   50  0001 C CNN "Digikey part number"
 	1    7200 4600
 	-1   0    0    1
@@
 F 0 "J13" H 7172 4880 50  0000 R CNN
 F 1 "Motor_5" H 7172 4971 50  0000 R CNN
-F 2 "Connector_PinHeader_2.54mm:PinHeader_1x03_P2.54mm_Vertical" H 7200 4950 50  0001 C CNN
+F 2 "Connector_Harwin:Harwin_LTek-Male_03_P2.00mm_Vertical" H 7200 4950 50  0001 C CNN
 F 3 "~" H 7200 4950 50  0001 C CNN
+F 4 "952-1070-5-ND‎" H 0   0   50  0001 C CNN "Digikey part number"
 	1    7200 4950
 	-1   0    0    1
@@
 F 0 "J14" H 7172 5230 50  0000 R CNN
 F 1 "Motor_6" H 7172 5321 50  0000 R CNN
-F 2 "Connector_PinHeader_2.54mm:PinHeader_1x03_P2.54mm_Vertical" H 7200 5300 50  0001 C CNN
+F 2 "Connector_Harwin:Harwin_LTek-Male_03_P2.00mm_Vertical" H 7200 5300 50  0001 C CNN
 F 3 "~" H 7200 5300 50  0001 C CNN
+F 4 "952-1070-5-ND‎" H 0   0   50  0001 C CNN "Digikey part number"
 	1    7200 5300
 	-1   0    0    1
@@
 F 0 "J15" H 7172 5580 50  0000 R CNN
 F 1 "Motor_7" H 7172 5671 50  0000 R CNN
-F 2 "Connector_PinHeader_2.54mm:PinHeader_1x03_P2.54mm_Vertical" H 7200 5650 50  0001 C CNN
+F 2 "Connector_Harwin:Harwin_LTek-Male_03_P2.00mm_Vertical" H 7200 5650 50  0001 C CNN
 F 3 "~" H 7200 5650 50  0001 C CNN
+F 4 "952-1070-5-ND‎" H 0   0   50  0001 C CNN "Digikey part number"
 	1    7200 5650
 	-1   0    0    1
@@
 F 0 "J16" H 7172 5930 50  0000 R CNN
 F 1 "Motor_8" H 7172 6021 50  0000 R CNN
-F 2 "Connector_PinHeader_2.54mm:PinHeader_1x03_P2.54mm_Vertical" H 7200 6000 50  0001 C CNN
+F 2 "Connector_Harwin:Harwin_LTek-Male_03_P2.00mm_Vertical" H 7200 6000 50  0001 C CNN
 F 3 "~" H 7200 6000 50  0001 C CNN
+F 4 "952-1070-5-ND‎" H 0   0   50  0001 C CNN "Digikey part number"
 	1    7200 6000
 	-1   0    0    1
