File: electrical/control board/control board.sch (KiCad schematic (older format))
At the start: 56 parts, among them J1 analog_extra, J10 Motor_2, J11 Motor_3, J12 Motor_4, J13 Motor_5, J14 Motor_6, J15 Motor_7, J16 Motor_8, J2 Programming_Header, J4 datamate_sensors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

Commit message: replaced sensor with BMI160
Parts:
- removed C15, C17, C18: 0.1uF, Capacitor_SMD:C_0603_1608Metric_Pad1.05x0.95mm_HandSolder, symbol Device:C_Small
- removed U7: ICM20648, footprints:ICM-20648, symbol custom_symbols:ICM20648
- added 10u1, 10u2: C_Small, symbol Device:C_Small
- added C? (x2): 100nF, symbol Device:C_Small
- added J3: USB_B, Connector_USB:USB_B_TE_5787834_Vertical, symbol Connector:USB_B
- added R? (x2): 10k, symbol Device:R_Small
- added U3: LD1117S33TR_SOT223, Package_TO_SOT_SMD:SOT-223-3_TabPin2, symbol Regulator_Linear:LD1117S33TR_SOT223
- added U?: BMI160, symbol custom_symbols:BMI160
Connections:
- wire segments 251 -> 259
- no-connect marks 15 -> 19
Other:
- note added: "ADD DECOUPLING CAPS"
- note added: "Not connected to +5V to avoid overcurrent\non USB port attempting to power odroid"
- note removed: "This ICM won't work. Find a new one that can be soldered"

Commit message: routed new acceleration sensor
Parts:
- C11, C12: renamed from C?; footprint (none) -> Capacitor_SMD:C_0603_1608Metric_Pad1.05x0.95mm_HandSolder
- R3, R4: renamed from R?; footprint (none) -> Resistor_SMD:R_0603_1608Metric_Pad1.05x0.95mm_HandSolder
- U5: renamed from U?; footprint (none) -> Package_LGA:LGA-14_3x2.5mm_P0.5mm_LayoutBorder3x4y
Changed lines of the file:
@@
 $EndComp
 $Comp
-L custom_symbols:BMI160 U?
+L custom_symbols:BMI160 U5
 U 1 1 5C5716BD
 P 10350 7700
-F 0 "U?" H 10350 7815 50  0000 C CNN
+F 0 "U5" H 10350 7815 50  0000 C CNN
 F 1 "BMI160" H 10350 7724 50  0000 C CNN
-F 2 "" H 10350 7700 50  0001 C CNN
+F 2 "Package_LGA:LGA-14_3x2.5mm_P0.5mm_LayoutBorder3x4y" H 10350 7700 50  0001 C CNN
 F 3 "" H 10350 7700 50  0001 C CNN
 	1    10350 7700
@@
 $EndComp
 $Comp
-L power:+3.3V #PWR?
+L power:+3.3V #PWR0151
 U 1 1 5C57182B
 P 10800 7750
-F 0 "#PWR?" H 10800 7600 50  0001 C CNN
+F 0 "#PWR0151" H 10800 7600 50  0001 C CNN
 F 1 "+3.3V" H 10815 7923 50  0000 C CNN
 F 2 "" H 10800 7750 50  0001 C CNN
@@
 $EndComp
 $Comp
-L power:+3.3V #PWR?
+L power:+3.3V #PWR0152
 U 1 1 5C5718C7
 P 9850 8150
-F 0 "#PWR?" H 9850 8000 50  0001 C CNN
+F 0 "#PWR0152" H 9850 8000 50  0001 C CNN
 F 1 "+3.3V" H 9865 8323 50  0000 C CNN
 F 2 "" H 9850 8150 50  0001 C CNN
@@
 $EndComp
 $Comp
-L power:GND #PWR?
+L power:GND #PWR0154
 U 1 1 5C57196A
 P 9850 8500
-F 0 "#PWR?" H 9850 8250 50  0001 C CNN
+F 0 "#PWR0154" H 9850 8250 50  0001 C CNN
 F 1 "GND" H 9855 8327 50  0000 C CNN
 F 2 "" H 9850 8500 50  0001 C CNN
@@
 ICM_SDA
 $Comp
-L power:+3.3V #PWR?
+L power:+3.3V #PWR0155
 U 1 1 5C5BB028
 P 10900 8100
-F 0 "#PWR?" H 10900 7950 50  0001 C CNN
+F 0 "#PWR0155" H 10900 7950 50  0001 C CNN
 F 1 "+3.3V" H 10915 8273 50  0000 C CNN
 F 2 "" H 10900 8100 50  0001 C CNN
@@
 	10700 8400 11100 8400
 $Comp
-L Device:R_Small R?
+L Device:R_Small R3
 U 1 1 5C605A61
 P 10700 8600
-F 0 "R?" H 10759 8646 50  0000 L CNN
+F 0 "R3" H 10759 8646 50  0000 L CNN
 F 1 "10k" H 10759 8555 50  0000 L CNN
-F 2 "" H 10700 8600 50  0001 C CNN
+F 2 "Resistor_SMD:R_0603_1608Metric_Pad1.05x0.95mm_HandSolder" H 10700 8600 50  0001 C CNN
 F 3 "~" H 10700 8600 50  0001 C CNN
 	1    10700 8600
@@
 $EndComp
 $Comp
-L Device:R_Small R?
+L Device:R_Small R4
 U 1 1 5C605B1B
 P 10900 8600
-F 0 "R?" H 10959 8646 50  0000 L CNN
+F 0 "R4" H 10959 8646 50  0000 L CNN
 F 1 "10k" H 10959 8555 50  0000 L CNN
-F 2 "" H 10900 8600 50  0001 C CNN
+F 2 "Resistor_SMD:R_0603_1608Metric_Pad1.05x0.95mm_HandSolder" H 10900 8600 50  0001 C CNN
 F 3 "~" H 10900 8600 50  0001 C CNN
 	1    10900 8600
@@
 Connection ~ 10700 8400
 $Comp
-L power:+3.3V #PWR?
+L power:+3.3V #PWR0157
 U 1 1 5C62B5FC
 P 11200 8700
-F 0 "#PWR?" H 11200 8550 50  0001 C CNN
+F 0 "#PWR0157" H 11200 8550 50  0001 C CNN
 F 1 "+3.3V" H 11215 8873 50  0000 C CNN
 F 2 "" H 11200 8700 50  0001 C CNN
@@
 	10900 8750 11200 8750
 $Comp
-L Device:C_Small C?
+L Device:C_Small C11
 U 1 1 5C653227
 P 9700 8300
-F 0 "C?" H 9792 8346 50  0000 L CNN
+F 0 "C11" H 9792 8346 50  0000 L CNN
 F 1 "100nF" H 9792 8255 50  0000 L CNN
-F 2 "" H 9700 8300 50  0001 C CNN
+F 2 "Capacitor_SMD:C_0603_1608Metric_Pad1.05x0.95mm_HandSolder" H 9700 8300 50  0001 C CNN
 F 3 "~" H 9700 8300 50  0001 C CNN
 	1    9700 8300
@@
 $EndComp
 $Comp
-L Device:C_Small C?
+L Device:C_Small C12
 U 1 1 5C653307
 P 11100 7900
-F 0 "C?" H 11192 7946 50  0000 L CNN
+F 0 "C12" H 11192 7946 50  0000 L CNN
 F 1 "100nF" H 11192 7855 50  0000 L CNN
-F 2 "" H 11100 7900 50  0001 C CNN
+F 2 "Capacitor_SMD:C_0603_1608Metric_Pad1.05x0.95mm_HandSolder" H 11100 7900 50  0001 C CNN
 F 3 "~" H 11100 7900 50  0001 C CNN
 	1    11100 7900
@@
 Connection ~ 10800 7800
 $Comp
-L power:GND #PWR?
+L power:GND #PWR0158
 U 1 1 5C6A8B59
 P 11100 8050
-F 0 "#PWR?" H 11100 7800 50  0001 C CNN
+F 0 "#PWR0158" H 11100 7800 50  0001 C CNN
 F 1 "GND" H 11105 7877 50  0000 C CNN
 F 2 "" H 11100 8050 50  0001 C CNN

Commit message: added usb port and linear regulator
Parts:
- J3: footprint Connector_USB:USB_B_TE_5787834_Vertical -> Connector_USB:USB_B_OST_USB-B1HSxx_Horizontal
Other:
- note added: "Consider adding switch instead"
- note removed: "ADD DECOUPLING CAPS"
Changed lines of the file:
@@
 F 0 "J3" H 8755 2317 50  0000 C CNN
 F 1 "USB_B" H 8755 2226 50  0000 C CNN
-F 2 "Connector_USB:USB_B_TE_5787834_Vertical" H 8850 1800 50  0001 C CNN
+F 2 "Connector_USB:USB_B_OST_USB-B1HSxx_Horizontal" H 8850 1800 50  0001 C CNN
 F 3 " ~" H 8850 1800 50  0001 C CNN
 	1    8700 1850
@@
 Wire Wire Line
 	10050 1650 9950 1650
-Text Notes 8900 1200 0    50   ~ 0
-ADD DECOUPLING CAPS
 $Comp
 L Device:C_Small 10u1
@@
 NoConn ~ 10700 8000
 NoConn ~ 10700 8100
+Text Notes 9100 2400 0    50   ~ 0
+Consider adding switch instead
 $EndSCHEMATC

Commit message: replaced humidity sensor with one that exists
Parts:
- removed C1: 0.1uF, Capacitor_SMD:C_0603_1608Metric_Pad1.05x0.95mm_HandSolder, symbol Device:C_Small
- removed C4: 1uF, Capacitor_SMD:C_0603_1608Metric_Pad1.05x0.95mm_HandSolder, symbol Device:C_Small
- removed R1, R2: 4.7k, Resistor_SMD:R_0603_1608Metric_Pad1.05x0.95mm_HandSolder, symbol Device:R_Small
- removed U2: HIH6031, Package_SO:SOIC-8-N7_3.9x4.9mm_P1.27mm, symbol hih6031:HIH6031
- added C?: .1uF, symbol Device:C_Small
- added C?: .22uF, symbol Device:C_Small
- added R? (x2): 2.2k, symbol Device:R_Small
- added U?: HIH6131-021, symbol custom_symbols:HIH6131-021
- U5: Digikey part number (none) -> 828-1089-1-ND
Connections:
- wire segments 259 -> 250
- no-connect marks 19 -> 20
Changed lines of the file:
@@
 USART1_RX
-$Comp
-L hih6031:HIH6031 U2
-U 1 1 5BE098FF
-P 2100 6600
-F 0 "U2" H 2100 7147 60  0000 C CNN
-F 1 "HIH6031" H 2100 7041 60  0000 C CNN
-F 2 "Package_SO:SOIC-8-N7_3.9x4.9mm_P1.27mm" H 2200 6550 60  0001 C CNN
-F 3 "" H 2200 6550 60  0001 C CNN
-F 4 "HIH7130-000-001CT-ND " H 0   0   50  0001 C CNN "Digikey part number"
-	1    2100 6600
-	1    0    0    -1
-$EndComp
 $Comp
 L custom_symbols:ADM3061 U6
@@
 Wire Wire Line
 	2000 4300 2350 4300
-Text Label 850  6500 0    50   ~ 0
+Text Label 2500 6800 0    50   ~ 0
 HIH_SCL
-Text Label 850  6600 0    50   ~ 0
+Text Label 2500 6900 0    50   ~ 0
 HIH_SDA
-NoConn ~ 2550 6500
-NoConn ~ 2550 6600
-$Comp
-L Device:C_Small C1
-U 1 1 5BE62B2C
-P 700 6250
-F 0 "C1" H 792 6296 50  0000 L CNN
-F 1 "0.1uF" H 792 6205 50  0000 L CNN
-F 2 "Capacitor_SMD:C_0603_1608Metric_Pad1.05x0.95mm_HandSolder" H 700 6250 50  0001 C CNN
-F 3 "~" H 700 6250 50  0001 C CNN
-F 4 "1276-1005-1-ND " H 0   0   50  0001 C CNN "Digikey part number"
-	1    700  6250
-	1    0    0    -1
-$EndComp
-$Comp
-L power:GND #PWR0134
-U 1 1 5BE62C5B
-P 700 6550
-F 0 "#PWR0134" H 700 6300 50  0001 C CNN
-F 1 "GND" H 705 6377 50  0000 C CNN
-F 2 "" H 700 6550 50  0001 C CNN
-F 3 "" H 700 6550 50  0001 C CNN
-	1    700  6550
-	1    0    0    -1
-$EndComp
-$Comp
-L power:+3.3V #PWR0135
-U 1 1 5BE73B22
-P 2550 6150
-F 0 "#PWR0135" H 2550 6000 50  0001 C CNN
-F 1 "+3.3V" H 2565 6323 50  0000 C CNN
-F 2 "" H 2550 6150 50  0001 C CNN
-F 3 "" H 2550 6150 50  0001 C CNN
-	1    2550 6150
-	1    0    0    -1
-$EndComp
-Wire Wire Line
-	2550 6150 2550 6250
-$Comp
-L Device:C_Small C4
-U 1 1 5BE7C931
-P 2750 6350
-F 0 "C4" H 2842 6396 50  0000 L CNN
-F 1 "1uF" H 2842 6305 50  0000 L CNN
-F 2 "Capacitor_SMD:C_0603_1608Metric_Pad1.05x0.95mm_HandSolder" H 2750 6350 50  0001 C CNN
-F 3 "~" H 2750 6350 50  0001 C CNN
-F 4 "1276-1102-1-ND" H 0   0   50  0001 C CNN "Digikey part number"
-	1    2750 6350
-	1    0    0    -1
-$EndComp
-$Comp
-L power:GND #PWR0136
-U 1 1 5BE7C9C0
-P 2750 6450
-F 0 "#PWR0136" H 2750 6200 50  0001 C CNN
-F 1 "GND" H 2755 6277 50  0000 C CNN
-F 2 "" H 2750 6450 50  0001 C CNN
-F 3 "" H 2750 6450 50  0001 C CNN
-	1    2750 6450
-	1    0    0    -1
-$EndComp
-Wire Wire Line
-	2750 6250 2550 6250
-Connection ~ 2550 6250
-Wire Wire Line
-	2550 6250 2550 6300
-Wire Wire Line
-	850  6500 1250 6500
-Wire Wire Line
-	850  6600 1200 6600
-Wire Wire Line
-	1650 6400 700  6400
-Wire Wire Line
-	700  6400 700  6550
-Wire Wire Line
-	700  6350 700  6400
-Connection ~ 700  6400
-Wire Wire Line
-	1650 6300 1100 6300
-Wire Wire Line
-	1100 6300 1100 6100
-Wire Wire Line
-	1100 6100 700  6100
-Wire Wire Line
-	700  6100 700  6150
-$Comp
-L Device:R_Small R1
-U 1 1 5BEC4A6B
-P 1500 6850
-F 0 "R1" V 1304 6850 50  0000 C CNN
-F 1 "4.7k" V 1395 6850 50  0000 C CNN
-F 2 "Resistor_SMD:R_0603_1608Metric_Pad1.05x0.95mm_HandSolder" H 1500 6850 50  0001 C CNN
-F 3 "~" H 1500 6850 50  0001 C CNN
-F 4 "CR0603-JW-472ELFCT-ND " H 0   0   50  0001 C CNN "Digikey part number"
-	1    1500 6850
-	0    1    1    0
-$EndComp
-$Comp
-L Device:R_Small R2
-U 1 1 5BEC4B58
-P 1500 7150
-F 0 "R2" V 1304 7150 50  0000 C CNN
-F 1 "4.7k" V 1395 7150 50  0000 C CNN
-F 2 "Resistor_SMD:R_0603_1608Metric_Pad1.05x0.95mm_HandSolder" H 1500 7150 50  0001 C CNN
-F 3 "~" H 1500 7150 50  0001 C CNN
-F 4 "CR0603-JW-472ELFCT-ND " H 0   0   50  0001 C CNN "Digikey part number"
-	1    1500 7150
-	0    1    1    0
-$EndComp
-Wire Wire Line
-	1400 6850 1250 6850
-Wire Wire Line
-	1250 6850 1250 6500
-Connection ~ 1250 6500
-Wire Wire Line
-	1250 6500 1650 6500
-Wire Wire Line
-	1400 7150 1200 7150
-Wire Wire Line
-	1200 7150 1200 6600
-Connection ~ 1200 6600
-Wire Wire Line
-	1200 6600 1650 6600
-$Comp
-L power:+3.3V #PWR0137
-U 1 1 5BED8178
-P 1900 6900
-F 0 "#PWR0137" H 1900 6750 50  0001 C CNN
-F 1 "+3.3V" H 1915 7073 50  0000 C CNN
-F 2 "" H 1900 6900 50  0001 C CNN
-F 3 "" H 1900 6900 50  0001 C CNN
-	1    1900 6900
-	1    0    0    -1
-$EndComp
-Wire Wire Line
-	1600 7150 1750 7150
-Wire Wire Line
-	1900 7150 1900 6900
-Wire Wire Line
-	1600 6850 1750 6850
-Wire Wire Line
-	1750 6850 1750 7150
-Connection ~ 1750 7150
-Wire Wire Line
-	1750 7150 1900 7150
-Text Notes 2500 7400 0    50   ~ 0
+Text Notes 1700 6100 0    50   ~ 0
 UART4 : Odroid\nUART2 : Motors\nUART1 : Sensors\nUART3 : Misc
 Text Label 5750 9550 0    50   ~ 0
@@
 F 2 "Package_LGA:LGA-14_3x2.5mm_P0.5mm_LayoutBorder3x4y" H 10350 7700 50  0001 C CNN
 F 3 "" H 10350 7700 50  0001 C CNN
+F 4 " 828-1089-1-ND" H 0   0   50  0001 C CNN "Digikey part number"
 	1    10350 7700
 	1    0    0    -1
@@
 Text Notes 9100 2400 0    50   ~ 0
 Consider adding switch instead
+$Comp
+L custom_symbols:HIH6131-021 U?
+U 1 1 5C781F5E
+P 1700 6700
+F 0 "U?" H 1700 6815 50  0000 C CNN
+F 1 "HIH6131-021" H 1700 6724 50  0000 C CNN
+F 2 "" H 1700 6700 50  0001 C CNN
+F 3 "" H 1700 6700 50  0001 C CNN
+	1    1700 6700
+	1    0    0    -1
+$EndComp
+NoConn ~ 1300 7100
+NoConn ~ 2100 7000
+NoConn ~ 2100 7100
+$Comp
+L power:+3.3V #PWR?
+U 1 1 5C7B592C
+P 1200 6700
+F 0 "#PWR?" H 1200 6550 50  0001 C CNN
+F 1 "+3.3V" H 1215 6873 50  0000 C CNN
+F 2 "" H 1200 6700 50  0001 C CNN
+F 3 "" H 1200 6700 50  0001 C CNN
+	1    1200 6700
+	1    0    0    -1
+$EndComp
+Wire Wire Line
+	1300 6800 1200 6800
+Wire Wire Line
+	1200 6800 1200 6700
+$Comp
+L Device:C_Small C?
+U 1 1 5C7C745D
+P 1150 6900
+F 0 "C?" V 921 6900 50  0000 C CNN
+F 1 ".1uF" V 1012 6900 50  0000 C CNN
+F 2 "" H 1150 6900 50  0001 C CNN
+F 3 "~" H 1150 6900 50  0001 C CNN
+	1    1150 6900
+	0    1    1    0
+$EndComp
+$Comp
+L Device:C_Small C?
+U 1 1 5C7C7CF9
+P 850 6900
+F 0 "C?" H 758 6854 50  0000 R CNN
+F 1 ".22uF" H 758 6945 50  0000 R CNN
+F 2 "" H 850 6900 50  0001 C CNN
+F 3 "~" H 850 6900 50  0001 C CNN
+	1    850  6900
+	-1   0    0    1
+$EndComp
+Wire Wire Line
+	1300 6900 1250 6900
+Wire Wire Line
+	850  6800 1000 6800
+Connection ~ 1200 6800
+Wire Wire Line
+	850  7000 1300 7000
+Wire Wire Line
+	1050 6900 1000 6900
+Wire Wire Line
+	1000 6900 1000 6800
+Connection ~ 1000 6800
+Wire Wire Line
+	1000 6800 1200 6800
+Wire Wire Line
+	2500 6800 2150 6800
+Wire Wire Line
+	2500 6900 2400 6900
+$Comp
+L Device:R_Small R?
+U 1 1 5C87269B
+P 2150 6600
+F 0 "R?" H 2209 6646 50  0000 L CNN
+F 1 "2.2k" H 2209 6555 50  0000 L CNN
+F 2 "" H 2150 6600 50  0001 C CNN
+F 3 "~" H 2150 6600 50  0001 C CNN
+	1    2150 6600
+	1    0    0    -1
+$EndComp
+$Comp
+L Device:R_Small R?
+U 1 1 5C87274D
+P 2400 6600
+F 0 "R?" H 2459 6646 50  0000 L CNN
+F 1 "2.2k" H 2459 6555 50  0000 L CNN
+F 2 "" H 2400 6600 50  0001 C CNN
+F 3 "~" H 2400 6600 50  0001 C CNN
+	1    2400 6600
+	1    0    0    -1
+$EndComp
+Wire Wire Line
+	2400 6700 2400 6900
+Connection ~ 2400 6900
+Wire Wire Line
+	2400 6900 2100 6900
+Wire Wire Line
+	2150 6700 2150 6800
+Connection ~ 2150 6800
+Wire Wire Line
+	2150 6800 2100 6800
+$Comp
+L power:+3.3V #PWR?
+U 1 1 5C89335F
+P 2150 6500
+F 0 "#PWR?" H 2150 6350 50  0001 C CNN
+F 1 "+3.3V" H 2165 6673 50  0000 C CNN
+F 2 "" H 2150 6500 50  0001 C CNN
+F 3 "" H 2150 6500 50  0001 C CNN
+	1    2150 6500
+	1    0    0    -1
+$EndComp
+$Comp
+L power:+3.3V #PWR?
+U 1 1 5C8933FB
+P 2400 6500
+F 0 "#PWR?" H 2400 6350 50  0001 C CNN
+F 1 "+3.3V" H 2415 6673 50  0000 C CNN
+F 2 "" H 2400 6500 50  0001 C CNN
+F 3 "" H 2400 6500 50  0001 C CNN
+	1    2400 6500
+	1    0    0    -1
+$EndComp
 $EndSCHEMATC

Commit message: mostly finished routing control board
Parts:
- C1, C4: renamed from C?; footprint (none) -> Capacitor_SMD:C_0603_1608Metric_Pad1.05x0.95mm_HandSolder
- R1, R2: renamed from R?; footprint (none) -> Resistor_SMD:R_0603_1608Metric_Pad1.05x0.95mm_HandSolder
- U2: renamed from U?; footprint (none) -> Package_SO:SOIC-8_3.9x4.9mm_P1.27mm
Changed lines of the file:
@@
 Consider adding switch instead
 $Comp
-L custom_symbols:HIH6131-021 U?
+L custom_symbols:HIH6131-021 U2
 U 1 1 5C781F5E
 P 1700 6700
-F 0 "U?" H 1700 6815 50  0000 C CNN
+F 0 "U2" H 1700 6815 50  0000 C CNN
 F 1 "HIH6131-021" H 1700 6724 50  0000 C CNN
-F 2 "" H 1700 6700 50  0001 C CNN
+F 2 "Package_SO:SOIC-8_3.9x4.9mm_P1.27mm" H 1700 6700 50  0001 C CNN
 F 3 "" H 1700 6700 50  0001 C CNN
 	1    1700 6700
@@
 NoConn ~ 2100 7100
 $Comp
-L power:+3.3V #PWR?
+L power:+3.3V #PWR0134
 U 1 1 5C7B592C
 P 1200 6700
-F 0 "#PWR?" H 1200 6550 50  0001 C CNN
+F 0 "#PWR0134" H 1200 6550 50  0001 C CNN
 F 1 "+3.3V" H 1215 6873 50  0000 C CNN
 F 2 "" H 1200 6700 50  0001 C CNN
@@
 	1200 6800 1200 6700
 $Comp
-L Device:C_Small C?
+L Device:C_Small C4
 U 1 1 5C7C745D
 P 1150 6900
-F 0 "C?" V 921 6900 50  0000 C CNN
+F 0 "C4" V 921 6900 50  0000 C CNN
 F 1 ".1uF" V 1012 6900 50  0000 C CNN
-F 2 "" H 1150 6900 50  0001 C CNN
+F 2 "Capacitor_SMD:C_0603_1608Metric_Pad1.05x0.95mm_HandSolder" H 1150 6900 50  0001 C CNN
 F 3 "~" H 1150 6900 50  0001 C CNN
 	1    1150 6900
@@
 $EndComp
 $Comp
-L Device:C_Small C?
+L Device:C_Small C1
 U 1 1 5C7C7CF9
 P 850 6900
-F 0 "C?" H 758 6854 50  0000 R CNN
+F 0 "C1" H 758 6854 50  0000 R CNN
 F 1 ".22uF" H 758 6945 50  0000 R CNN
-F 2 "" H 850 6900 50  0001 C CNN
+F 2 "Capacitor_SMD:C_0603_1608Metric_Pad1.05x0.95mm_HandSolder" H 850 6900 50  0001 C CNN
 F 3 "~" H 850 6900 50  0001 C CNN
 	1    850  6900
@@
 	2500 6900 2400 6900
 $Comp
-L Device:R_Small R?
+L Device:R_Small R1
 U 1 1 5C87269B
 P 2150 6600
-F 0 "R?" H 2209 6646 50  0000 L CNN
+F 0 "R1" H 2209 6646 50  0000 L CNN
 F 1 "2.2k" H 2209 6555 50  0000 L CNN
-F 2 "" H 2150 6600 50  0001 C CNN
+F 2 "Resistor_SMD:R_0603_1608Metric_Pad1.05x0.95mm_HandSolder" H 2150 6600 50  0001 C CNN
 F 3 "~" H 2150 6600 50  0001 C CNN
 	1    2150 6600
@@
 $EndComp
 $Comp
-L Device:R_Small R?
+L Device:R_Small R2
 U 1 1 5C87274D
 P 2400 6600
-F 0 "R?" H 2459 6646 50  0000 L CNN
+F 0 "R2" H 2459 6646 50  0000 L CNN
 F 1 "2.2k" H 2459 6555 50  0000 L CNN
-F 2 "" H 2400 6600 50  0001 C CNN
+F 2 "Resistor_SMD:R_0603_1608Metric_Pad1.05x0.95mm_HandSolder" H 2400 6600 50  0001 C CNN
 F 3 "~" H 2400 6600 50  0001 C CNN
 	1    2400 6600
@@
 	2150 6800 2100 6800
 $Comp
-L power:+3.3V #PWR?
+L power:+3.3V #PWR0135
 U 1 1 5C89335F
 P 2150 6500
-F 0 "#PWR?" H 2150 6350 50  0001 C CNN
+F 0 "#PWR0135" H 2150 6350 50  0001 C CNN
 F 1 "+3.3V" H 2165 6673 50  0000 C CNN
 F 2 "" H 2150 6500 50  0001 C CNN
@@
 $EndComp
 $Comp
-L power:+3.3V #PWR?
+L power:+3.3V #PWR0136
 U 1 1 5C8933FB
 P 2400 6500
-F 0 "#PWR?" H 2400 6350 50  0001 C CNN
+F 0 "#PWR0136" H 2400 6350 50  0001 C CNN
 F 1 "+3.3V" H 2415 6673 50  0000 C CNN
 F 2 "" H 2400 6500 50  0001 C CNN

Commit message: added capacitors to linear regulator
Parts:
- C15: renamed from 10u1; value C_Small -> 10uF; footprint (none) -> Capacitor_SMD:C_0603_1608Metric_Pad1.05x0.95mm_HandSolder
- C16: renamed from 10u2; value C_Small -> 10uF; footprint (none) -> Capacitor_SMD:C_0603_1608Metric_Pad1.05x0.95mm_HandSolder
Changed lines of the file:
@@
 	10050 1650 9950 1650
 $Comp
-L Device:C_Small 10u1
+L Device:C_Small C15
 U 1 1 5C449EA8
 P 9100 1750
-F 0 "10u1" H 9192 1796 50  0000 L CNN
-F 1 "C_Small" H 9192 1705 50  0000 L CNN
-F 2 "" H 9100 1750 50  0001 C CNN
+F 0 "C15" H 9192 1796 50  0000 L CNN
+F 1 "10uF" H 9192 1705 50  0000 L CNN
+F 2 "Capacitor_SMD:C_0603_1608Metric_Pad1.05x0.95mm_HandSolder" H 9100 1750 50  0001 C CNN
 F 3 "~" H 9100 1750 50  0001 C CNN
 	1    9100 1750
@@
 	9100 1650 9200 1650
 $Comp
-L Device:C_Small 10u2
+L Device:C_Small C16
 U 1 1 5C44A03D
 P 9950 1750
-F 0 "10u2" H 10042 1796 50  0000 L CNN
-F 1 "C_Small" H 10042 1705 50  0000 L CNN
-F 2 "" H 9950 1750 50  0001 C CNN
+F 0 "C16" H 10042 1796 50  0000 L CNN
+F 1 "10uF" H 10042 1705 50  0000 L CNN
+F 2 "Capacitor_SMD:C_0603_1608Metric_Pad1.05x0.95mm_HandSolder" H 9950 1750 50  0001 C CNN
 F 3 "~" H 9950 1750 50  0001 C CNN
 	1    9950 1750

Commit message: Added pads to access internal layers
Parts:
- added J8: Power_Header, footprints:1x2 individual header, symbol Connector:Conn_01x02_Male
Connections:
- wire segments 250 -> 254
Changed lines of the file:
@@
 	1    0    0    -1
 $EndComp
+$Comp
+L Connector:Conn_01x02_Male J8
+U 1 1 5C8CEA72
+P 9200 3850
+F 0 "J8" H 9172 3730 50  0000 R CNN
+F 1 "Power_Header" H 9172 3821 50  0000 R CNN
+F 2 "footprints:1x2 individual header" H 9200 3850 50  0001 C CNN
+F 3 "~" H 9200 3850 50  0001 C CNN
+	1    9200 3850
+	-1   0    0    1
+$EndComp
+$Comp
+L power:+3.3V #PWR0137
+U 1 1 5C8CEE3C
+P 8900 3700
+F 0 "#PWR0137" H 8900 3550 50  0001 C CNN
+F 1 "+3.3V" H 8915 3873 50  0000 C CNN
+F 2 "" H 8900 3700 50  0001 C CNN
+F 3 "" H 8900 3700 50  0001 C CNN
+	1    8900 3700
+	1    0    0    -1
+$EndComp
+$Comp
+L power:GND #PWR0159
+U 1 1 5C8CEEE1
+P 8900 3900
+F 0 "#PWR0159" H 8900 3650 50  0001 C CNN
+F 1 "GND" H 8905 3727 50  0000 C CNN
+F 2 "" H 8900 3900 50  0001 C CNN
+F 3 "" H 8900 3900 50  0001 C CNN
+	1    8900 3900
+	1    0    0    -1
+$EndComp
+Wire Wire Line
+	9000 3750 8900 3750
+Wire Wire Line
+	8900 3750 8900 3700
+Wire Wire Line
+	9000 3850 8900 3850
+Wire Wire Line
+	8900 3850 8900 3900
 $EndSCHEMATC

Commit message: added reset button
Parts:
- added C17: .1uF, Capacitor_SMD:C_0603_1608Metric_Pad1.05x0.95mm_HandSolder, symbol Device:C_Small
- added C18: 2.2uF, Capacitor_SMD:C_0603_1608Metric_Pad1.05x0.95mm_HandSolder, symbol Device:C_Small
- added SW1: SW_Push, Button_Switch_SMD:SW_SPST_PTS645, symbol Switch:SW_Push
Connections:
- wire segments 254 -> 264
Changed lines of the file:
@@
 Connection ~ 2300 2000
 Wire Wire Line
-	2300 2000 1600 2000
+	2300 2000 1850 2000
 $Comp
 L power:GND #PWR0156
@@
 Wire Wire Line
 	8900 3850 8900 3900
+$Comp
+L Device:C_Small C17
+U 1 1 5C8F21D2
+P 1850 2100
+F 0 "C17" H 1942 2146 50  0000 L CNN
+F 1 ".1uF" H 1942 2055 50  0000 L CNN
+F 2 "Capacitor_SMD:C_0603_1608Metric_Pad1.05x0.95mm_HandSolder" H 1850 2100 50  0001 C CNN
+F 3 "~" H 1850 2100 50  0001 C CNN
+	1    1850 2100
+	1    0    0    -1
+$EndComp
+Connection ~ 1850 2000
+Wire Wire Line
+	1850 2000 1600 2000
+$Comp
+L power:GND #PWR0160
+U 1 1 5C8F2473
+P 1850 2250
+F 0 "#PWR0160" H 1850 2000 50  0001 C CNN
+F 1 "GND" H 1855 2077 50  0000 C CNN
+F 2 "" H 1850 2250 50  0001 C CNN
+F 3 "" H 1850 2250 50  0001 C CNN
+	1    1850 2250
+	1    0    0    -1
+$EndComp
+Wire Wire Line
+	1850 2200 1850 2250
+$Comp
+L power:GND #PWR0161
+U 1 1 5C903FD4
+P 2250 2250
+F 0 "#PWR0161" H 2250 2000 50  0001 C CNN
+F 1 "GND" H 2255 2077 50  0000 C CNN
+F 2 "" H 2250 2250 50  0001 C CNN
+F 3 "" H 2250 2250 50  0001 C CNN
+	1    2250 2250
+	1    0    0    -1
+$EndComp
+$Comp
+L Device:C_Small C18
+U 1 1 5C904082
+P 2300 2550
+F 0 "C18" H 2392 2596 50  0000 L CNN
+F 1 "2.2uF" H 2392 2505 50  0000 L CNN
+F 2 "Capacitor_SMD:C_0603_1608Metric_Pad1.05x0.95mm_HandSolder" H 2300 2550 50  0001 C CNN
+F 3 "~" H 2300 2550 50  0001 C CNN
+	1    2300 2550
+	1    0    0    -1
+$EndComp
+$Comp
+L power:GND #PWR0162
+U 1 1 5C904295
+P 2300 2700
+F 0 "#PWR0162" H 2300 2450 50  0001 C CNN
+F 1 "GND" H 2305 2527 50  0000 C CNN
+F 2 "" H 2300 2700 50  0001 C CNN
+F 3 "" H 2300 2700 50  0001 C CNN
+	1    2300 2700
+	1    0    0    -1
+$EndComp
+Wire Wire Line
+	2300 2700 2300 2650
+Wire Wire Line
+	2350 2400 2300 2400
+Wire Wire Line
+	2300 2400 2300 2450
+Wire Wire Line
+	2250 2250 2250 2200
+Wire Wire Line
+	2250 2200 2350 2200
+$Comp
+L Switch:SW_Push SW1
+U 1 1 5C93AE21
+P 1400 1200
+F 0 "SW1" H 1400 1485 50  0000 C CNN
+F 1 "SW_Push" H 1400 1394 50  0000 C CNN
+F 2 "Button_Switch_SMD:SW_SPST_PTS645" H 1400 1400 50  0001 C CNN
+F 3 "" H 1400 1400 50  0001 C CNN
+F 4 "PTS645SM43SMTR92 LFS " H 0   0   50  0001 C CNN "Digikey part number"
+	1    1400 1200
+	1    0    0    -1
+$EndComp
+Text Label 1000 1200 0    50   ~ 0
+NRST
+$Comp
+L power:GND #PWR0163
+U 1 1 5C93AFA3
+P 1650 1250
+F 0 "#PWR0163" H 1650 1000 50  0001 C CNN
+F 1 "GND" H 1655 1077 50  0000 C CNN
+F 2 "" H 1650 1250 50  0001 C CNN
+F 3 "" H 1650 1250 50  0001 C CNN
+	1    1650 1250
+	1    0    0    -1
+$EndComp
+Wire Wire Line
+	1650 1250 1650 1200
+Wire Wire Line
+	1650 1200 1600 1200
+Wire Wire Line
+	1200 1200 1000 1200
 $EndSCHEMATC
