File: electrical/control board/control board.sch (KiCad schematic (older format))
At the start: 68 parts, among them J1 analog_extra, J10 Motor_2, J11 Motor_3, J12 Motor_4, J13 Motor_5, J14 Motor_6, J15 Motor_7, J16 Motor_8, J17 USB_to_5V, J18 Storage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

Commit message: Added power leds and bugfixes
Parts:
- added D?: LED-YELLOW, LED_SMD:LED_0603_1608Metric_Pad1.05x0.95mm_HandSolder, symbol Device:LED
- added D?: LED-GREEN, LED_SMD:LED_0603_1608Metric_Pad1.05x0.95mm_HandSolder, symbol Device:LED
- added R? (x2): 220, Resistor_SMD:R_0603_1608Metric_Pad1.05x0.95mm_HandSolder, symbol Device:R_Small
Connections:
- wire segments 275 -> 287
Changed lines of the file:
@@
 Connection ~ 1200 6800
 Wire Wire Line
-	850  7000 1300 7000
+	850  7000 1050 7000
 Wire Wire Line
 	1050 6900 1000 6900
@@
 Wire Wire Line
 	9150 1200 9150 1050
+$Comp
+L power:GND #PWR?
+U 1 1 5C621FD8
+P 1050 7100
+F 0 "#PWR?" H 1050 6850 50  0001 C CNN
+F 1 "GND" H 1055 6927 50  0000 C CNN
+F 2 "" H 1050 7100 50  0001 C CNN
+F 3 "" H 1050 7100 50  0001 C CNN
+	1    1050 7100
+	1    0    0    -1
+$EndComp
+Connection ~ 1050 7000
+Wire Wire Line
+	1050 7000 1300 7000
+Wire Wire Line
+	1050 7000 1050 7100
+$Comp
+L Device:R_Small R?
+U 1 1 5C638A1B
+P 5600 3700
+F 0 "R?" V 5796 3700 50  0000 C CNN
+F 1 "220" V 5705 3700 50  0000 C CNN
+F 2 "Resistor_SMD:R_0603_1608Metric_Pad1.05x0.95mm_HandSolder" H 5600 3700 50  0001 C CNN
+F 3 "~" H 5600 3700 50  0001 C CNN
+F 4 "A130087CT-ND" H 50  950 50  0001 C CNN "Digikey part number"
+	1    5600 3700
+	0    -1   -1   0
+$EndComp
+$Comp
+L Device:LED D?
+U 1 1 5C638BA8
+P 5250 3700
+F 0 "D?" H 5241 3916 50  0000 C CNN
+F 1 "LED-YELLOW" H 5241 3825 50  0000 C CNN
+F 2 "LED_SMD:LED_0603_1608Metric_Pad1.05x0.95mm_HandSolder" H 5250 3700 50  0001 C CNN
+F 3 "http://optoelectronics.liteon.com/upload/download/DS22-2000-224/LTST-C191KSKT.PDF" H 5250 3700 50  0001 C CNN
+F 4 "160-1448-1-ND " H 50  950 50  0001 C CNN "Digikey part number"
+	1    5250 3700
+	1    0    0    -1
+$EndComp
+Wire Wire Line
+	5500 3700 5400 3700
+$Comp
+L power:GND #PWR?
+U 1 1 5C64E1EA
+P 5000 3800
+F 0 "#PWR?" H 5000 3550 50  0001 C CNN
+F 1 "GND" H 5005 3627 50  0000 C CNN
+F 2 "" H 5000 3800 50  0001 C CNN
+F 3 "" H 5000 3800 50  0001 C CNN
+	1    5000 3800
+	1    0    0    -1
+$EndComp
+$Comp
+L power:+3.3V #PWR?
+U 1 1 5C64E2BB
+P 5850 3650
+F 0 "#PWR?" H 5850 3500 50  0001 C CNN
+F 1 "+3.3V" H 5865 3823 50  0000 C CNN
+F 2 "" H 5850 3650 50  0001 C CNN
+F 3 "" H 5850 3650 50  0001 C CNN
+	1    5850 3650
+	1    0    0    -1
+$EndComp
+Wire Wire Line
+	5850 3650 5850 3700
+Wire Wire Line
+	5850 3700 5700 3700
+Wire Wire Line
+	5100 3700 5000 3700
+Wire Wire Line
+	5000 3700 5000 3800
+$Comp
+L Device:LED D?
+U 1 1 5C679AE8
+P 5250 4150
+F 0 "D?" H 5241 4366 50  0000 C CNN
+F 1 "LED-GREEN" H 5241 4275 50  0000 C CNN
+F 2 "LED_SMD:LED_0603_1608Metric_Pad1.05x0.95mm_HandSolder" H 5250 4150 50  0001 C CNN
+F 3 "http://optoelectronics.liteon.com/upload/download/DS22-2000-228/LTST-C191KGKT.PDF" H 5250 4150 50  0001 C CNN
+F 4 "160-1446-1-ND " H 50  1050 50  0001 C CNN "Digikey part number"
+	1    5250 4150
+	1    0    0    -1
+$EndComp
+$Comp
+L Device:R_Small R?
+U 1 1 5C679E35
+P 5600 4150
+F 0 "R?" V 5796 4150 50  0000 C CNN
+F 1 "220" V 5705 4150 50  0000 C CNN
+F 2 "Resistor_SMD:R_0603_1608Metric_Pad1.05x0.95mm_HandSolder" H 5600 4150 50  0001 C CNN
+F 3 "~" H 5600 4150 50  0001 C CNN
+F 4 "A130087CT-ND" H 50  1400 50  0001 C CNN "Digikey part number"
+	1    5600 4150
+	0    -1   -1   0
+$EndComp
+$Comp
+L power:+5V #PWR?
+U 1 1 5C67A019
+P 5850 4100
+F 0 "#PWR?" H 5850 3950 50  0001 C CNN
+F 1 "+5V" H 5865 4273 50  0000 C CNN
+F 2 "" H 5850 4100 50  0001 C CNN
+F 3 "" H 5850 4100 50  0001 C CNN
+	1    5850 4100
+	1    0    0    -1
+$EndComp
+$Comp
+L power:GND #PWR?
+U 1 1 5C67A11A
+P 5000 4200
+F 0 "#PWR?" H 5000 3950 50  0001 C CNN
+F 1 "GND" H 5005 4027 50  0000 C CNN
+F 2 "" H 5000 4200 50  0001 C CNN
+F 3 "" H 5000 4200 50  0001 C CNN
+	1    5000 4200
+	1    0    0    -1
+$EndComp
+Wire Wire Line
+	5100 4150 5000 4150
+Wire Wire Line
+	5000 4150 5000 4200
+Wire Wire Line
+	5400 4150 5500 4150
+Wire Wire Line
+	5700 4150 5850 4150
+Wire Wire Line
+	5850 4150 5850 4100
 $EndSCHEMATC

Commit message: Added power indicators
Parts:
- gave numbers to parts that had none: 4
Changed lines of the file:
@@
 	9150 1200 9150 1050
 $Comp
-L power:GND #PWR?
+L power:GND #PWR0166
 U 1 1 5C621FD8
 P 1050 7100
-F 0 "#PWR?" H 1050 6850 50  0001 C CNN
+F 0 "#PWR0166" H 1050 6850 50  0001 C CNN
 F 1 "GND" H 1055 6927 50  0000 C CNN
 F 2 "" H 1050 7100 50  0001 C CNN
@@
 	1050 7000 1050 7100
 $Comp
-L Device:R_Small R?
+L Device:R_Small R5
 U 1 1 5C638A1B
 P 5600 3700
-F 0 "R?" V 5796 3700 50  0000 C CNN
+F 0 "R5" V 5796 3700 50  0000 C CNN
 F 1 "220" V 5705 3700 50  0000 C CNN
 F 2 "Resistor_SMD:R_0603_1608Metric_Pad1.05x0.95mm_HandSolder" H 5600 3700 50  0001 C CNN
@@
 $EndComp
 $Comp
-L Device:LED D?
+L Device:LED D7
 U 1 1 5C638BA8
 P 5250 3700
-F 0 "D?" H 5241 3916 50  0000 C CNN
+F 0 "D7" H 5241 3916 50  0000 C CNN
 F 1 "LED-YELLOW" H 5241 3825 50  0000 C CNN
 F 2 "LED_SMD:LED_0603_1608Metric_Pad1.05x0.95mm_HandSolder" H 5250 3700 50  0001 C CNN
@@
 	5500 3700 5400 3700
 $Comp
-L power:GND #PWR?
+L power:GND #PWR0167
 U 1 1 5C64E1EA
 P 5000 3800
-F 0 "#PWR?" H 5000 3550 50  0001 C CNN
+F 0 "#PWR0167" H 5000 3550 50  0001 C CNN
 F 1 "GND" H 5005 3627 50  0000 C CNN
 F 2 "" H 5000 3800 50  0001 C CNN
@@
 $EndComp
 $Comp
-L power:+3.3V #PWR?
+L power:+3.3V #PWR0168
 U 1 1 5C64E2BB
 P 5850 3650
-F 0 "#PWR?" H 5850 3500 50  0001 C CNN
+F 0 "#PWR0168" H 5850 3500 50  0001 C CNN
 F 1 "+3.3V" H 5865 3823 50  0000 C CNN
 F 2 "" H 5850 3650 50  0001 C CNN
@@
 	5000 3700 5000 3800
 $Comp
-L Device:LED D?
+L Device:LED D8
 U 1 1 5C679AE8
 P 5250 4150
-F 0 "D?" H 5241 4366 50  0000 C CNN
+F 0 "D8" H 5241 4366 50  0000 C CNN
 F 1 "LED-GREEN" H 5241 4275 50  0000 C CNN
 F 2 "LED_SMD:LED_0603_1608Metric_Pad1.05x0.95mm_HandSolder" H 5250 4150 50  0001 C CNN
@@
 $EndComp
 $Comp
-L Device:R_Small R?
+L Device:R_Small R6
 U 1 1 5C679E35
 P 5600 4150
-F 0 "R?" V 5796 4150 50  0000 C CNN
+F 0 "R6" V 5796 4150 50  0000 C CNN
 F 1 "220" V 5705 4150 50  0000 C CNN
 F 2 "Resistor_SMD:R_0603_1608Metric_Pad1.05x0.95mm_HandSolder" H 5600 4150 50  0001 C CNN
@@
 $EndComp
 $Comp
-L power:+5V #PWR?
+L power:+5V #PWR0169
 U 1 1 5C67A019
 P 5850 4100
-F 0 "#PWR?" H 5850 3950 50  0001 C CNN
+F 0 "#PWR0169" H 5850 3950 50  0001 C CNN
 F 1 "+5V" H 5865 4273 50  0000 C CNN
 F 2 "" H 5850 4100 50  0001 C CNN
@@
 $EndComp
 $Comp
-L power:GND #PWR?
+L power:GND #PWR0170
 U 1 1 5C67A11A
 P 5000 4200
-F 0 "#PWR?" H 5000 3950 50  0001 C CNN
+F 0 "#PWR0170" H 5000 3950 50  0001 C CNN
 F 1 "GND" H 5005 4027 50  0000 C CNN
 F 2 "" H 5000 4200 50  0001 C CNN

Commit message: Added 24V measurement
Parts:
- added R12: 100k, Resistor_SMD:R_0603_1608Metric_Pad1.05x0.95mm_HandSolder, symbol Device:R_Small
- added R20: 6.6k, Resistor_SMD:R_0603_1608Metric_Pad1.05x0.95mm_HandSolder, symbol Device:R_Small
Connections:
- net labels added: 24V_MEASURE
- wire segments 287 -> 290
Changed lines of the file:
@@
 L Device:R_Small R15
 U 1 1 5BFDA6B2
-P 5200 6800
-F 0 "R15" H 5259 6846 50  0000 L CNN
-F 1 "100k" H 5259 6755 50  0000 L CNN
-F 2 "Resistor_SMD:R_0603_1608Metric_Pad1.05x0.95mm_HandSolder" H 5200 6800 50  0001 C CNN
-F 3 "~" H 5200 6800 50  0001 C CNN
-F 4 "CR0603-JW-104ELFCT-ND" H 0   0   50  0001 C CNN "Digikey part number"
-	1    5200 6800
+P 5850 6800
+F 0 "R15" H 5909 6846 50  0000 L CNN
+F 1 "100k" H 5909 6755 50  0000 L CNN
+F 2 "Resistor_SMD:R_0603_1608Metric_Pad1.05x0.95mm_HandSolder" H 5850 6800 50  0001 C CNN
+F 3 "~" H 5850 6800 50  0001 C CNN
+F 4 "CR0603-JW-104ELFCT-ND" H 650 0   50  0001 C CNN "Digikey part number"
+	1    5850 6800
 	1    0    0    -1
 $EndComp
@@
 L Device:R_Small R16
 U 1 1 5BFDA748
-P 5200 7150
-F 0 "R16" H 5259 7196 50  0000 L CNN
-F 1 "3.6k" H 5259 7105 50  0000 L CNN
-F 2 "Resistor_SMD:R_0603_1608Metric_Pad1.05x0.95mm_HandSolder" H 5200 7150 50  0001 C CNN
-F 3 "~" H 5200 7150 50  0001 C CNN
-F 4 "RMCF0603JT3K60CT-ND" H 0   0   50  0001 C CNN "Digikey part number"
-	1    5200 7150
+P 5850 7150
+F 0 "R16" H 5909 7196 50  0000 L CNN
+F 1 "3.6k" H 5909 7105 50  0000 L CNN
+F 2 "Resistor_SMD:R_0603_1608Metric_Pad1.05x0.95mm_HandSolder" H 5850 7150 50  0001 C CNN
+F 3 "~" H 5850 7150 50  0001 C CNN
+F 4 "RMCF0603JT3K60CT-ND" H 650 0   50  0001 C CNN "Digikey part number"
+	1    5850 7150
 	1    0    0    -1
 $EndComp
@@
 L power:GND #PWR0140
 U 1 1 5C002DD8
-P 5200 7250
-F 0 "#PWR0140" H 5200 7000 50  0001 C CNN
-F 1 "GND" H 5205 7077 50  0000 C CNN
-F 2 "" H 5200 7250 50  0001 C CNN
-F 3 "" H 5200 7250 50  0001 C CNN
-	1    5200 7250
+P 5850 7250
+F 0 "#PWR0140" H 5850 7000 50  0001 C CNN
+F 1 "GND" H 5855 7077 50  0000 C CNN
+F 2 "" H 5850 7250 50  0001 C CNN
+F 3 "" H 5850 7250 50  0001 C CNN
+	1    5850 7250
 	1    0    0    -1
 $EndComp
@@
 L power:+48V #PWR0143
 U 1 1 5C003142
-P 5200 6700
-F 0 "#PWR0143" H 5200 6550 50  0001 C CNN
-F 1 "+48V" H 5215 6873 50  0000 C CNN
-F 2 "" H 5200 6700 50  0001 C CNN
-F 3 "" H 5200 6700 50  0001 C CNN
-	1    5200 6700
+P 5850 6700
+F 0 "#PWR0143" H 5850 6550 50  0001 C CNN
+F 1 "+48V" H 5865 6873 50  0000 C CNN
+F 2 "" H 5850 6700 50  0001 C CNN
+F 3 "" H 5850 6700 50  0001 C CNN
+	1    5850 6700
 	1    0    0    -1
 $EndComp
@@
 Text Label 4100 6950 0    50   ~ 0
 5V_MEASURE
-Text Label 4650 6950 0    50   ~ 0
+Text Label 5300 6950 0    50   ~ 0
 48V_MEASURE
 Wire Wire Line
-	4650 6950 5200 6950
-Wire Wire Line
-	5200 6900 5200 6950
-Connection ~ 5200 6950
-Wire Wire Line
-	5200 6950 5200 7050
+	5300 6950 5850 6950
+Wire Wire Line
+	5850 6900 5850 6950
+Connection ~ 5850 6950
+Wire Wire Line
+	5850 6950 5850 7050
 Wire Wire Line
 	4100 6950 4600 6950
@@
 Wire Wire Line
 	4050 6950 4050 7050
-Wire Notes Line
-	3400 6350 5500 6350
-Wire Notes Line
-	5500 6350 5500 7600
-Wire Notes Line
-	5500 7600 3400 7600
 Wire Notes Line
 	3400 7600 3400 6350
@@
 Wire Wire Line
 	5850 4150 5850 4100
+$Comp
+L Device:R_Small R12
+U 1 1 5C6D5458
+P 5250 6800
+F 0 "R12" H 5309 6846 50  0000 L CNN
+F 1 "100k" H 5309 6755 50  0000 L CNN
+F 2 "Resistor_SMD:R_0603_1608Metric_Pad1.05x0.95mm_HandSolder" H 5250 6800 50  0001 C CNN
+F 3 "~" H 5250 6800 50  0001 C CNN
+F 4 "CR0603-JW-104ELFCT-ND" H 0   0   50  0001 C CNN "Digikey part number"
+	1    5250 6800
+	1    0    0    -1
+$EndComp
+$Comp
+L Device:R_Small R20
+U 1 1 5C6D5658
+P 5250 7150
+F 0 "R20" H 5309 7196 50  0000 L CNN
+F 1 "6.6k" H 5309 7105 50  0000 L CNN
+F 2 "Resistor_SMD:R_0603_1608Metric_Pad1.05x0.95mm_HandSolder" H 5250 7150 50  0001 C CNN
+F 3 "~" H 5250 7150 50  0001 C CNN
+F 4 "A129698CT-ND" H 0   0   50  0001 C CNN "Digikey part number"
+	1    5250 7150
+	1    0    0    -1
+$EndComp
+$Comp
+L power:GND #PWR0171
+U 1 1 5C6D5D2C
+P 5250 7250
+F 0 "#PWR0171" H 5250 7000 50  0001 C CNN
+F 1 "GND" H 5255 7077 50  0000 C CNN
+F 2 "" H 5250 7250 50  0001 C CNN
+F 3 "" H 5250 7250 50  0001 C CNN
+	1    5250 7250
+	1    0    0    -1
+$EndComp
+$Comp
+L power:+24V #PWR0172
+U 1 1 5C6D5DF7
+P 5250 6700
+F 0 "#PWR0172" H 5250 6550 50  0001 C CNN
+F 1 "+24V" H 5265 6873 50  0000 C CNN
+F 2 "" H 5250 6700 50  0001 C CNN
+F 3 "" H 5250 6700 50  0001 C CNN
+	1    5250 6700
+	1    0    0    -1
+$EndComp
+Wire Wire Line
+	5250 6900 5250 6950
+Text Label 4700 6950 0    50   ~ 0
+24V_MEASURE
+Wire Wire Line
+	4700 6950 5250 6950
+Connection ~ 5250 6950
+Wire Wire Line
+	5250 6950 5250 7050
+Wire Notes Line
+	6150 6350 6150 7600
+Wire Notes Line
+	3400 6350 6150 6350
+Wire Notes Line
+	3400 7600 6150 7600
+Text Label 3750 3800 0    50   ~ 0
+24V_MEASURE
 $EndSCHEMATC

Commit message: Found parts
Parts:
- R10, R11, R17, R18, R19, R5, R9: value 220 -> 68; Digikey part number A130087CT-ND -> RMCF0603JT68R0CT-ND
- R6: value 220 -> 180; Digikey part number A130087CT-ND -> (none)
Changed lines of the file:
@@
 P 4750 1650
 F 0 "R11" V 4554 1650 50  0000 C CNN
-F 1 "220" V 4645 1650 50  0000 C CNN
+F 1 "68" V 4645 1650 50  0000 C CNN
 F 2 "Resistor_SMD:R_0603_1608Metric_Pad1.05x0.95mm_HandSolder" H 4750 1650 50  0001 C CNN
 F 3 "~" H 4750 1650 50  0001 C CNN
-F 4 "A130087CT-ND" H 0   0   50  0001 C CNN "Digikey part number"
+F 4 "RMCF0603JT68R0CT-ND" H 0   0   50  0001 C CNN "Digikey part number"
 	1    4750 1650
 	0    1    1    0
@@
 P 4750 1300
 F 0 "R10" V 4554 1300 50  0000 C CNN
-F 1 "220" V 4645 1300 50  0000 C CNN
+F 1 "68" V 4645 1300 50  0000 C CNN
 F 2 "Resistor_SMD:R_0603_1608Metric_Pad1.05x0.95mm_HandSolder" H 4750 1300 50  0001 C CNN
 F 3 "~" H 4750 1300 50  0001 C CNN
-F 4 "A130087CT-ND" H 0   0   50  0001 C CNN "Digikey part number"
+F 4 "RMCF0603JT68R0CT-ND" H 0   0   50  0001 C CNN "Digikey part number"
 	1    4750 1300
 	0    1    1    0
@@
 P 4750 900
 F 0 "R9" V 4946 900 50  0000 C CNN
-F 1 "220" V 4855 900 50  0000 C CNN
+F 1 "68" V 4855 900 50  0000 C CNN
 F 2 "Resistor_SMD:R_0603_1608Metric_Pad1.05x0.95mm_HandSolder" H 4750 900 50  0001 C CNN
 F 3 "~" H 4750 900 50  0001 C CNN
-F 4 "A130087CT-ND" H 0   0   50  0001 C CNN "Digikey part number"
+F 4 "RMCF0603JT68R0CT-ND" H 0   0   50  0001 C CNN "Digikey part number"
 	1    4750 900
 	0    -1   -1   0
@@
 P 5550 3100
 F 0 "R19" V 5746 3100 50  0000 C CNN
-F 1 "220" V 5655 3100 50  0000 C CNN
+F 1 "68" V 5655 3100 50  0000 C CNN
 F 2 "Resistor_SMD:R_0603_1608Metric_Pad1.05x0.95mm_HandSolder" H 5550 3100 50  0001 C CNN
 F 3 "~" H 5550 3100 50  0001 C CNN
-F 4 "A130087CT-ND" H 0   0   50  0001 C CNN "Digikey part number"
+F 4 "RMCF0603JT68R0CT-ND" H 0   0   50  0001 C CNN "Digikey part number"
 	1    5550 3100
 	0    -1   -1   0
@@
 P 5550 2750
 F 0 "R18" V 5746 2750 50  0000 C CNN
-F 1 "220" V 5655 2750 50  0000 C CNN
+F 1 "68" V 5655 2750 50  0000 C CNN
 F 2 "Resistor_SMD:R_0603_1608Metric_Pad1.05x0.95mm_HandSolder" H 5550 2750 50  0001 C CNN
 F 3 "~" H 5550 2750 50  0001 C CNN
-F 4 "A130087CT-ND" H 0   0   50  0001 C CNN "Digikey part number"
+F 4 "RMCF0603JT68R0CT-ND" H 0   0   50  0001 C CNN "Digikey part number"
 	1    5550 2750
 	0    -1   -1   0
@@
 P 5550 2350
 F 0 "R17" V 5746 2350 50  0000 C CNN
-F 1 "220" V 5655 2350 50  0000 C CNN
+F 1 "68" V 5655 2350 50  0000 C CNN
 F 2 "Resistor_SMD:R_0603_1608Metric_Pad1.05x0.95mm_HandSolder" H 5550 2350 50  0001 C CNN
 F 3 "~" H 5550 2350 50  0001 C CNN
-F 4 "A130087CT-ND" H 0   0   50  0001 C CNN "Digikey part number"
+F 4 "RMCF0603JT68R0CT-ND" H 0   0   50  0001 C CNN "Digikey part number"
 	1    5550 2350
 	0    -1   -1   0
@@
 P 5600 3700
 F 0 "R5" V 5796 3700 50  0000 C CNN
-F 1 "220" V 5705 3700 50  0000 C CNN
+F 1 "68" V 5705 3700 50  0000 C CNN
 F 2 "Resistor_SMD:R_0603_1608Metric_Pad1.05x0.95mm_HandSolder" H 5600 3700 50  0001 C CNN
 F 3 "~" H 5600 3700 50  0001 C CNN
-F 4 "A130087CT-ND" H 50  950 50  0001 C CNN "Digikey part number"
+F 4 "RMCF0603JT68R0CT-ND" H 50  950 50  0001 C CNN "Digikey part number"
 	1    5600 3700
 	0    -1   -1   0
@@
 P 5600 4150
 F 0 "R6" V 5796 4150 50  0000 C CNN
-F 1 "220" V 5705 4150 50  0000 C CNN
+F 1 "180" V 5705 4150 50  0000 C CNN
 F 2 "Resistor_SMD:R_0603_1608Metric_Pad1.05x0.95mm_HandSolder" H 5600 4150 50  0001 C CNN
 F 3 "~" H 5600 4150 50  0001 C CNN
-F 4 "A130087CT-ND" H 50  1400 50  0001 C CNN "Digikey part number"
+F 4 "~" H 50  1400 50  0001 C CNN "Digikey part number"
 	1    5600 4150
 	0    -1   -1   0

Commit message: Fixed trace seperatation
Parts:
- U5: footprint Package_LGA:LGA-14_3x2.5mm_P0.5mm_LayoutBorder3x4y -> footprints:LGA-14_3x2.5mm_P0.5mm_pads_shrunk
Changed lines of the file:
@@
 F 0 "U5" H 10350 7815 50  0000 C CNN
 F 1 "BMI160" H 10350 7724 50  0000 C CNN
-F 2 "Package_LGA:LGA-14_3x2.5mm_P0.5mm_LayoutBorder3x4y" H 10350 7700 50  0001 C CNN
+F 2 "footprints:LGA-14_3x2.5mm_P0.5mm_pads_shrunk" H 10350 7700 50  0001 C CNN
 F 3 "" H 10350 7700 50  0001 C CNN
 F 4 "828-1057-1-ND" H 0   0   50  0001 C CNN "Digikey part number"

Commit message: tweaked silkscreen and re-exported gerbers
Other:
- note added: "Add 120 Ohm resistors across data lines?\n"
Changed lines of the file:
@@
 Text Label 3750 3800 0    50   ~ 0
 24V_MEASURE
+Text Notes 5800 9100 0    50   ~ 0
+Add 120 Ohm resistors across data lines?\n
 $EndSCHEMATC
