File: electrical/control board power/control board power.sch (KiCad schematic (older format))
At the start: 24 parts

Commit message: made a mess, then fixed it
Parts:
- removed C? (x2): 10uF, Capacitor_SMD:C_0603_1608Metric_Pad1.05x0.95mm_HandSolder, symbol Device:C_Small
- removed C? (x2): 1uF, Capacitor_SMD:C_0603_1608Metric_Pad1.05x0.95mm_HandSolder, symbol Device:C_Small
- removed C?: 10pF, Capacitor_SMD:C_0603_1608Metric_Pad1.05x0.95mm_HandSolder, symbol Device:C_Small
- removed C? (x2): .1uF, Capacitor_SMD:C_0603_1608Metric_Pad1.05x0.95mm_HandSolder, symbol Device:C_Small
- removed C?: 2.2nF, Capacitor_SMD:C_0603_1608Metric_Pad1.05x0.95mm_HandSolder, symbol Device:C_Small
- removed C?: 100pF, Capacitor_SMD:C_0603_1608Metric_Pad1.05x0.95mm_HandSolder, symbol Device:C_Small
- removed C? (x2): 22uF, Capacitor_SMD:C_0603_1608Metric_Pad1.05x0.95mm_HandSolder, symbol Device:C_Small
- removed C? (x2): 4.7uF, Capacitor_SMD:C_0603_1608Metric_Pad1.05x0.95mm_HandSolder, symbol Device:C_Small
- removed J?: 48V_IN, Connector_PinHeader_2.54mm:PinHeader_1x02_P2.54mm_Vertical, symbol Connector_Generic:Conn_01x02
- removed J?: Barrel_Jack, symbol Connector:Barrel_Jack
- removed J?: 5V, Connector_PinHeader_2.54mm:PinHeader_1x02_P2.54mm_Vertical, symbol Connector_Generic:Conn_01x02
- removed L? (x2): 33uH, Inductor_THT:L_Radial_D12.0mm_P6.00mm_MuRATA_1900R, symbol Device:L_Small
- removed R?: 4.02k, Resistor_SMD:R_0603_1608Metric_Pad1.05x0.95mm_HandSolder, symbol Device:R_Small
- removed R?: 100k, Resistor_SMD:R_0603_1608Metric_Pad1.05x0.95mm_HandSolder, symbol Device:R_Small
- removed R?: 5.11k, Resistor_SMD:R_0603_1608Metric_Pad1.05x0.95mm_HandSolder, symbol Device:R_Small
- removed U?: LD1117S33TR_SOT223, Package_TO_SOT_SMD:SOT-223-3_TabPin2, symbol Regulator_Linear:LD1117S33TR_SOT223
- removed U? (x2): LTC7103-LT7103, footprints:LTC7103, symbol custom_symbols:LTC7103-LT7103
Connections:
- net labels removed: +12V, +3.3V, +48V, +5V, 48V_IN, GND
- wire segments 140 -> 0
- no-connect marks 8 -> 0
Other:
- note removed: "Check regulator is correct voltage"
- note removed: "DO NOT CONNECT 12V AND 48V SIMUTANIOUSLY!!!!"
- note removed: "Power"

Commit message: transfered power section to a new project
for real this time
Parts:
- added C? (x2): 10uF, Capacitor_SMD:C_0603_1608Metric_Pad1.05x0.95mm_HandSolder, symbol Device:C_Small
- added C? (x2): 1uF, Capacitor_SMD:C_0603_1608Metric_Pad1.05x0.95mm_HandSolder, symbol Device:C_Small
- added C?: 10pF, Capacitor_SMD:C_0603_1608Metric_Pad1.05x0.95mm_HandSolder, symbol Device:C_Small
- added C? (x2): .1uF, Capacitor_SMD:C_0603_1608Metric_Pad1.05x0.95mm_HandSolder, symbol Device:C_Small
- added C?: 2.2nF, Capacitor_SMD:C_0603_1608Metric_Pad1.05x0.95mm_HandSolder, symbol Device:C_Small
- added C?: 100pF, Capacitor_SMD:C_0603_1608Metric_Pad1.05x0.95mm_HandSolder, symbol Device:C_Small
- added C? (x2): 22uF, Capacitor_SMD:C_0603_1608Metric_Pad1.05x0.95mm_HandSolder, symbol Device:C_Small
- added C? (x2): 4.7uF, Capacitor_SMD:C_0603_1608Metric_Pad1.05x0.95mm_HandSolder, symbol Device:C_Small
- added D? (x3): LED, symbol Device:LED
- added J?: 48V_IN, Connector_PinHeader_2.54mm:PinHeader_1x02_P2.54mm_Vertical, symbol Connector_Generic:Conn_01x02
- added J?: Barrel_Jack, symbol Connector:Barrel_Jack
- added J?: 5V, Connector_PinHeader_2.54mm:PinHeader_1x02_P2.54mm_Vertical, symbol Connector_Generic:Conn_01x02
- added L? (x2): 33uH, Inductor_THT:L_Radial_D12.0mm_P6.00mm_MuRATA_1900R, symbol Device:L_Small
- added R? (x3): R_Small, Resistor_SMD:R_0603_1608Metric_Pad1.05x0.95mm_HandSolder, symbol Device:R_Small
- added R?: 4.02k, Resistor_SMD:R_0603_1608Metric_Pad1.05x0.95mm_HandSolder, symbol Device:R_Small
- added R?: 100k, Resistor_SMD:R_0603_1608Metric_Pad1.05x0.95mm_HandSolder, symbol Device:R_Small
- added R?: 5.11k, Resistor_SMD:R_0603_1608Metric_Pad1.05x0.95mm_HandSolder, symbol Device:R_Small
- added U?: LD1117S33TR_SOT223, Package_TO_SOT_SMD:SOT-223-3_TabPin2, symbol Regulator_Linear:LD1117S33TR_SOT223
- added U? (x2): LTC7103-LT7103, footprints:LTC7103, symbol custom_symbols:LTC7103-LT7103
Connections:
- net labels added: +12V, +3.3V, +48V, +5V, 48V_IN, GND
- wire segments 0 -> 155
- no-connect marks 0 -> 8
Other:
- note added: "Check regulator is correct voltage"
- note added: "DO NOT CONNECT 12V AND 48V SIMUTANIOUSLY!!!!"
- note added: "Power"
- note added: "Power Indicators"

Commit message: Moved current measurement to power board
Parts:
- added C?: C_Small, Capacitor_SMD:C_0603_1608Metric_Pad1.05x0.95mm_HandSolder, symbol Device:C_Small
- added R?: 1m, footprints:FC4L64, symbol Device:R_Shunt
- added U?: INA240-INA240, Package_SO:TSSOP-8_4.4x3mm_P0.65mm, symbol custom_symbols:INA240-INA240
Connections:
- net labels added: CURRENT_MEASURE
- wire segments 155 -> 170
Other:
- moved on the sheet: U?

Commit message: added low side switches to control board power
Parts:
- added J?: Power_Connector, Connector_Molex:Molex_Mini-Fit_Jr_5566-08A2_2x04_P4.20mm_Vertical, symbol Connector_Generic:Conn_02x04_Counter_Clockwise
- added J?: Conn_01x08, Connector_PinHeader_2.54mm:PinHeader_1x08_P2.54mm_Vertical, symbol Connector_Generic:Conn_01x08
- added Q? (x4): Q_NMOS_GDS, symbol Device:Q_NMOS_GDS
- added R? (x4): 10k, Resistor_SMD:R_0603_1608Metric_Pad1.05x0.95mm_HandSolder, symbol Device:R_Small
Connections:
- net labels added: +24V, SWITCH_A, SWITCH_B, SWITCH_C, SWITCH_D
- wire segments 170 -> 231
Other:
- note added: "Consider moving to power board"
- moved on the sheet: U?

Commit message: made a footprint with long pads and a hole in the middle
Parts:
- added J5: Conn_01x05, Connector_PinHeader_2.54mm:PinHeader_1x05_P2.54mm_Vertical, symbol Connector_Generic:Conn_01x05
- D1, D2, D3: renamed from D?; footprint (none) -> LED_SMD:LED_0603_1608Metric_Pad1.05x0.95mm_HandSolder
- U2, U3: renamed from U?; footprint footprints:LTC7103 -> footprints:LTC7103_long_pads_hole
- gave numbers to parts that had none: 38
Connections:
- wire segments 231 -> 237

Commit message: fixed the mess
Other:
- note added: "Check capacitor voltage ratings!!!"
- note added: "Look at Connor's 5V converter board to check component ratings, etc."
Changed lines of the file:
@@
 Wire Wire Line
 	5500 10400 5500 10450
+Text Notes 3250 1350 0    50   ~ 0
+Check capacitor voltage ratings!!!
+Text Notes 4950 1150 0    50   ~ 0
+Look at Connor's 5V converter board to check component ratings, etc.
 $EndSCHEMATC

Commit message: found a part for the barrel jack
Parts:
- J3: footprint (none) -> PJ-002AH:CUI_PJ-002AH; Digikey part number (none) -> CP-002AH-ND
Changed lines of the file:
@@
 F 0 "J3" H 2355 5575 50  0000 C CNN
 F 1 "Barrel_Jack" H 2355 5484 50  0000 C CNN
-F 2 "" H 2350 5210 50  0001 C CNN
+F 2 "PJ-002AH:CUI_PJ-002AH" H 2350 5210 50  0001 C CNN
 F 3 "~" H 2350 5210 50  0001 C CNN
+F 4 "CP-002AH-ND " H 0   0   50  0001 C CNN "Digikey part number"
 	1    2300 5250
 	1    0    0    -1
@@
 L Connector_Generic:Conn_01x05 J5
 U 1 1 5C361B4D
-P 5750 10200
-F 0 "J5" H 5830 10242 50  0000 L CNN
-F 1 "Conn_01x05" H 5830 10151 50  0000 L CNN
-F 2 "Connector_PinHeader_2.54mm:PinHeader_1x05_P2.54mm_Vertical" H 5750 10200 50  0001 C CNN
-F 3 "~" H 5750 10200 50  0001 C CNN
-	1    5750 10200
-	1    0    0    -1
-$EndComp
-Text Label 5150 10000 0    50   ~ 0
+P 7250 8100
+F 0 "J5" H 7330 8142 50  0000 L CNN
+F 1 "Conn_01x05" H 7330 8051 50  0000 L CNN
+F 2 "Connector_PinHeader_2.54mm:PinHeader_1x05_P2.54mm_Vertical" H 7250 8100 50  0001 C CNN
+F 3 "~" H 7250 8100 50  0001 C CNN
+	1    7250 8100
+	1    0    0    -1
+$EndComp
+Text Label 6650 7900 0    50   ~ 0
 SWITCH_A
-Text Label 5150 10100 0    50   ~ 0
+Text Label 6650 8000 0    50   ~ 0
 SWITCH_B
-Text Label 5150 10300 0    50   ~ 0
+Text Label 6650 8200 0    50   ~ 0
 SWITCH_D
-Text Label 5150 10200 0    50   ~ 0
+Text Label 6650 8100 0    50   ~ 0
 SWITCH_C
 Wire Wire Line
-	5550 10000 5150 10000
-Wire Wire Line
-	5550 10100 5150 10100
-Wire Wire Line
-	5550 10200 5150 10200
-Wire Wire Line
-	5550 10300 5150 10300
+	7050 7900 6650 7900
+Wire Wire Line
+	7050 8000 6650 8000
+Wire Wire Line
+	7050 8100 6650 8100
+Wire Wire Line
+	7050 8200 6650 8200
 $Comp
 L power:GND #PWR0138
 U 1 1 5C399CC8
-P 5500 10450
-F 0 "#PWR0138" H 5500 10200 50  0001 C CNN
-F 1 "GND" H 5505 10277 50  0000 C CNN
-F 2 "" H 5500 10450 50  0001 C CNN
-F 3 "" H 5500 10450 50  0001 C CNN
-	1    5500 10450
-	1    0    0    -1
-$EndComp
-Wire Wire Line
-	5550 10400 5500 10400
-Wire Wire Line
-	5500 10400 5500 10450
+P 7000 8350
+F 0 "#PWR0138" H 7000 8100 50  0001 C CNN
+F 1 "GND" H 7005 8177 50  0000 C CNN
+F 2 "" H 7000 8350 50  0001 C CNN
+F 3 "" H 7000 8350 50  0001 C CNN
+	1    7000 8350
+	1    0    0    -1
+$EndComp
+Wire Wire Line
+	7050 8300 7000 8300
+Wire Wire Line
+	7000 8300 7000 8350
 Text Notes 3250 1350 0    50   ~ 0
 Check capacitor voltage ratings!!!

Commit message: found parts for most of the stuff on the control board
Other:
- note added: "Unnessesary"
- note removed: "Consider moving to power board"
Changed lines of the file:
@@
 Wire Wire Line
 	5350 8000 5350 7900
-Text Notes 1850 10000 0    50   ~ 0
-Consider moving to power board
 $Comp
 L Connector_Generic:Conn_02x04_Counter_Clockwise J6
@@
 Text Notes 4950 1150 0    50   ~ 0
 Look at Connor's 5V converter board to check component ratings, etc.
+Wire Notes Line
+	750  7650 8050 7650
+Wire Notes Line
+	8050 7650 8050 10800
+Wire Notes Line
+	8050 10800 750  10800
+Wire Notes Line
+	750  10800 750  7650
+Text Notes 5500 10350 0    50   ~ 0
+Unnessesary
 $EndSCHEMATC
