File: electrical/control board power/control board power.sch (KiCad schematic (older format))
At the start: 54 parts, among them J1 48V_IN, J10 48V_from_conversion, J11 MOTOR_2, J12 MOTOR_6, J13 MOTOR_3, J14 MOTOR_7, J15 MOTOR_4, J16 MOTOR_8, J2 5V, J3 Barrel_Jack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

Commit message: changed footprint for motor headers
Parts:
- removed J9: 24V_from_conversion, Connector_Molex:Molex_Mini-Fit_Jr_5566-08A2_2x04_P4.20mm_Vertical, symbol Connector_Generic:Conn_02x04_Odd_Even
- added J9: 24V_from_conversion, Connector_Molex:Molex_Mini-Fit_Jr_5566-08A2_2x04_P4.20mm_Vertical, symbol Connector_Generic:Conn_02x04_Top_Bottom
- J11, J12, J13, J14, J15, J16, J7, J8: footprint Connector_Molex:Molex_Mini-Fit_Jr_5566-02A2_2x01_P4.20mm_Vertical -> Connector_Molex:Molex_Mini-Fit_Sr_42819-22XX_1x02_P10.00mm_Vertical_ThermalVias
Other:
- note added: "check current rating on headers!"
Changed lines of the file:
@@
 	11800 5200 11800 5100
-$Comp
-L Connector_Generic:Conn_02x04_Odd_Even J9
-U 1 1 5C602E58
-P 12000 5950
-F 0 "J9" H 12050 6267 50  0000 C CNN
-F 1 "24V_from_conversion" H 12050 6176 50  0000 C CNN
-F 2 "Connector_Molex:Molex_Mini-Fit_Jr_5566-08A2_2x04_P4.20mm_Vertical" H 12000 5950 50  0001 C CNN
-F 3 "~" H 12000 5950 50  0001 C CNN
-	1    12000 5950
-	1    0    0    -1
-$EndComp
 $Comp
 L power:GND #PWR0140
@@
 F 0 "J7" H 11329 7342 50  0000 L CNN
 F 1 "MOTOR_1" H 11329 7251 50  0000 L CNN
-F 2 "Connector_Molex:Molex_Mini-Fit_Jr_5566-02A2_2x01_P4.20mm_Vertical" H 11250 7350 50  0001 C CNN
+F 2 "Connector_Molex:Molex_Mini-Fit_Sr_42819-22XX_1x02_P10.00mm_Vertical_ThermalVias" H 11250 7350 50  0001 C CNN
 F 3 "~" H 11250 7350 50  0001 C CNN
 	1    11250 7350
@@
 F 0 "J11" H 12179 7342 50  0000 L CNN
 F 1 "MOTOR_2" H 12179 7251 50  0000 L CNN
-F 2 "Connector_Molex:Molex_Mini-Fit_Jr_5566-02A2_2x01_P4.20mm_Vertical" H 12100 7350 50  0001 C CNN
+F 2 "Connector_Molex:Molex_Mini-Fit_Sr_42819-22XX_1x02_P10.00mm_Vertical_ThermalVias" H 12100 7350 50  0001 C CNN
 F 3 "~" H 12100 7350 50  0001 C CNN
 	1    12100 7350
@@
 F 0 "J13" H 13029 7342 50  0000 L CNN
 F 1 "MOTOR_3" H 13029 7251 50  0000 L CNN
-F 2 "Connector_Molex:Molex_Mini-Fit_Jr_5566-02A2_2x01_P4.20mm_Vertical" H 12950 7350 50  0001 C CNN
+F 2 "Connector_Molex:Molex_Mini-Fit_Sr_42819-22XX_1x02_P10.00mm_Vertical_ThermalVias" H 12950 7350 50  0001 C CNN
 F 3 "~" H 12950 7350 50  0001 C CNN
 	1    12950 7350
@@
 F 0 "J15" H 13879 7342 50  0000 L CNN
 F 1 "MOTOR_4" H 13879 7251 50  0000 L CNN
-F 2 "Connector_Molex:Molex_Mini-Fit_Jr_5566-02A2_2x01_P4.20mm_Vertical" H 13800 7350 50  0001 C CNN
+F 2 "Connector_Molex:Molex_Mini-Fit_Sr_42819-22XX_1x02_P10.00mm_Vertical_ThermalVias" H 13800 7350 50  0001 C CNN
 F 3 "~" H 13800 7350 50  0001 C CNN
 	1    13800 7350
@@
 F 0 "J8" H 11329 8242 50  0000 L CNN
 F 1 "MOTOR_5" H 11329 8151 50  0000 L CNN
-F 2 "Connector_Molex:Molex_Mini-Fit_Jr_5566-02A2_2x01_P4.20mm_Vertical" H 11250 8250 50  0001 C CNN
+F 2 "Connector_Molex:Molex_Mini-Fit_Sr_42819-22XX_1x02_P10.00mm_Vertical_ThermalVias" H 11250 8250 50  0001 C CNN
 F 3 "~" H 11250 8250 50  0001 C CNN
 	1    11250 8250
@@
 F 0 "J12" H 12179 8242 50  0000 L CNN
 F 1 "MOTOR_6" H 12179 8151 50  0000 L CNN
-F 2 "Connector_Molex:Molex_Mini-Fit_Jr_5566-02A2_2x01_P4.20mm_Vertical" H 12100 8250 50  0001 C CNN
+F 2 "Connector_Molex:Molex_Mini-Fit_Sr_42819-22XX_1x02_P10.00mm_Vertical_ThermalVias" H 12100 8250 50  0001 C CNN
 F 3 "~" H 12100 8250 50  0001 C CNN
 	1    12100 8250
@@
 F 0 "J14" H 13029 8242 50  0000 L CNN
 F 1 "MOTOR_7" H 13029 8151 50  0000 L CNN
-F 2 "Connector_Molex:Molex_Mini-Fit_Jr_5566-02A2_2x01_P4.20mm_Vertical" H 12950 8250 50  0001 C CNN
+F 2 "Connector_Molex:Molex_Mini-Fit_Sr_42819-22XX_1x02_P10.00mm_Vertical_ThermalVias" H 12950 8250 50  0001 C CNN
 F 3 "~" H 12950 8250 50  0001 C CNN
 	1    12950 8250
@@
 F 0 "J16" H 13879 8242 50  0000 L CNN
 F 1 "MOTOR_8" H 13879 8151 50  0000 L CNN
-F 2 "Connector_Molex:Molex_Mini-Fit_Jr_5566-02A2_2x01_P4.20mm_Vertical" H 13800 8250 50  0001 C CNN
+F 2 "Connector_Molex:Molex_Mini-Fit_Sr_42819-22XX_1x02_P10.00mm_Vertical_ThermalVias" H 13800 8250 50  0001 C CNN
 F 3 "~" H 13800 8250 50  0001 C CNN
 	1    13800 8250
@@
 Wire Wire Line
 	13550 8350 13550 8500
+$Comp
+L Connector_Generic:Conn_02x04_Top_Bottom J9
+U 1 1 5C7111A9
+P 12000 5950
+F 0 "J9" H 12050 6267 50  0000 C CNN
+F 1 "24V_from_conversion" H 12050 6176 50  0000 C CNN
+F 2 "Connector_Molex:Molex_Mini-Fit_Jr_5566-08A2_2x04_P4.20mm_Vertical" H 12000 5950 50  0001 C CNN
+F 3 "~" H 12000 5950 50  0001 C CNN
+	1    12000 5950
+	1    0    0    -1
+$EndComp
+Text Notes 11900 8800 0    50   ~ 0
+check current rating on headers!
 $EndSCHEMATC

Commit message: stuff
Parts:
- removed J1: 48V_IN, Connector_PinHeader_2.54mm:PinHeader_1x02_P2.54mm_Vertical, symbol Connector_Generic:Conn_01x02
- removed J4: Conn_01x08, Connector_PinHeader_2.54mm:PinHeader_1x08_P2.54mm_Vertical, symbol Connector_Generic:Conn_01x08
- added J17: Switch_B, Connector_Molex:Molex_Nano-Fit_105309-xx02_1x02_P2.50mm_Vertical, symbol Connector_Generic:Conn_01x02
- added J18: Switch_C, Connector_Molex:Molex_Nano-Fit_105309-xx02_1x02_P2.50mm_Vertical, symbol Connector_Generic:Conn_01x02
- added J19: Switch_D, Connector_Molex:Molex_Nano-Fit_105309-xx02_1x02_P2.50mm_Vertical, symbol Connector_Generic:Conn_01x02
- added J4: Switch_A, Connector_Molex:Molex_Nano-Fit_105309-xx02_1x02_P2.50mm_Vertical, symbol Connector_Generic:Conn_01x02
- J10: footprint Connector_Molex:Molex_Mini-Fit_Jr_5566-02A2_2x01_P4.20mm_Vertical -> Connector_Molex:Molex_Mini-Fit_Jr_5566-02A_2x01_P4.20mm_Vertical
- J11, J12, J13, J14, J15, J16, J7, J8: footprint Connector_Molex:Molex_Mini-Fit_Sr_42819-22XX_1x02_P10.00mm_Vertical_ThermalVias -> Connector_Molex:Molex_Mini-Fit_Sr_42819-22XX_1x02_P10.00mm_Vertical
- J5: value Conn_01x05 -> Switch_Input; footprint Connector_PinHeader_2.54mm:PinHeader_1x05_P2.54mm_Vertical -> Connector_Harwin:Harwin_LTek-Male_05_P2.00mm_Vertical
Connections:
- wire segments 292 -> 288
Changed lines of the file:
@@
 	1    0    0    -1
 $EndComp
-Text Label 1100 4750 0    50   ~ 0
-48V_IN
 Text Notes 1000 5600 0    50   ~ 0
 Power
@@
 F 3 "http://www.st.com/st-web-ui/static/active/en/resource/technical/document/datasheet/CD00000544.pdf" H 2250 3650 50  0001 C CNN
 	1    2150 3900
-	1    0    0    -1
-$EndComp
-Wire Wire Line
-	1100 4950 1100 5050
-Wire Wire Line
-	1150 4950 1100 4950
-Wire Wire Line
-	1100 4850 1100 4750
-Wire Wire Line
-	1150 4850 1100 4850
-$Comp
-L power:GND #PWR0114
-U 1 1 5BC5881D
-P 1100 5050
-F 0 "#PWR0114" H 1100 4800 50  0001 C CNN
-F 1 "GND" H 1105 4877 50  0000 C CNN
-F 2 "" H 1100 5050 50  0001 C CNN
-F 3 "" H 1100 5050 50  0001 C CNN
-	1    1100 5050
-	1    0    0    -1
-$EndComp
-$Comp
-L Connector_Generic:Conn_01x02 J1
-U 1 1 5BC5876F
-P 1350 4850
-F 0 "J1" H 1429 4842 50  0000 L CNN
-F 1 "48V_IN" H 1429 4751 50  0000 L CNN
-F 2 "Connector_PinHeader_2.54mm:PinHeader_1x02_P2.54mm_Vertical" H 1350 4850 50  0001 C CNN
-F 3 "~" H 1350 4850 50  0001 C CNN
-	1    1350 4850
 	1    0    0    -1
 $EndComp
@@
 	1    0    0    -1
 $EndComp
-Text Notes 1300 4650 0    50   ~ 0
-DO NOT CONNECT 12V AND 48V SIMUTANIOUSLY!!!!
 Wire Notes Line
 	3600 5700 800  5700
@@
 	1500 9750 1950 9750
 Connection ~ 1950 9750
-Wire Wire Line
-	4800 9000 4800 8700
-$Comp
-L Connector_Generic:Conn_01x08 J4
-U 1 1 5C6CB645
-P 5750 8300
-F 0 "J4" H 5830 8292 50  0000 L CNN
-F 1 "Conn_01x08" H 5830 8201 50  0000 L CNN
-F 2 "Connector_PinHeader_2.54mm:PinHeader_1x08_P2.54mm_Vertical" H 5750 8300 50  0001 C CNN
-F 3 "~" H 5750 8300 50  0001 C CNN
-	1    5750 8300
-	1    0    0    -1
-$EndComp
-Wire Wire Line
-	5550 8700 4800 8700
-Wire Wire Line
-	5550 8500 3850 8500
-Wire Wire Line
-	3850 8500 3850 9000
-Wire Wire Line
-	2900 8300 2900 9000
-Wire Wire Line
-	2900 8300 5550 8300
-Wire Wire Line
-	5550 8100 1950 8100
-Wire Wire Line
-	1950 8100 1950 9000
-$Comp
-L power:+48V #PWR0132
-U 1 1 5C7AFDDB
-P 5350 7900
-F 0 "#PWR0132" H 5350 7750 50  0001 C CNN
-F 1 "+48V" H 5365 8073 50  0000 C CNN
-F 2 "" H 5350 7900 50  0001 C CNN
-F 3 "" H 5350 7900 50  0001 C CNN
-	1    5350 7900
-	1    0    0    -1
-$EndComp
-Wire Wire Line
-	5550 8600 5350 8600
-Wire Wire Line
-	5350 8600 5350 8400
-Wire Wire Line
-	5550 8400 5350 8400
-Connection ~ 5350 8400
-Wire Wire Line
-	5350 8400 5350 8200
-Wire Wire Line
-	5550 8200 5350 8200
-Connection ~ 5350 8200
-Wire Wire Line
-	5350 8200 5350 8000
-Wire Wire Line
-	5550 8000 5350 8000
-Connection ~ 5350 8000
-Wire Wire Line
-	5350 8000 5350 7900
 $Comp
 L Connector_Generic:Conn_02x04_Counter_Clockwise J6
@@
 P 7250 8100
 F 0 "J5" H 7330 8142 50  0000 L CNN
-F 1 "Conn_01x05" H 7330 8051 50  0000 L CNN
-F 2 "Connector_PinHeader_2.54mm:PinHeader_1x05_P2.54mm_Vertical" H 7250 8100 50  0001 C CNN
+F 1 "Switch_Input" H 7330 8051 50  0000 L CNN
+F 2 "Connector_Harwin:Harwin_LTek-Male_05_P2.00mm_Vertical" H 7250 8100 50  0001 C CNN
 F 3 "~" H 7250 8100 50  0001 C CNN
 	1    7250 8100
@@
 F 0 "J10" H 12179 5192 50  0000 L CNN
 F 1 "48V_from_conversion" H 12179 5101 50  0000 L CNN
-F 2 "Connector_Molex:Molex_Mini-Fit_Jr_5566-02A2_2x01_P4.20mm_Vertical" H 12100 5200 50  0001 C CNN
+F 2 "Connector_Molex:Molex_Mini-Fit_Jr_5566-02A_2x01_P4.20mm_Vertical" H 12100 5200 50  0001 C CNN
 F 3 "~" H 12100 5200 50  0001 C CNN
 	1    12100 5200
@@
 F 0 "J7" H 11329 7342 50  0000 L CNN
 F 1 "MOTOR_1" H 11329 7251 50  0000 L CNN
-F 2 "Connector_Molex:Molex_Mini-Fit_Sr_42819-22XX_1x02_P10.00mm_Vertical_ThermalVias" H 11250 7350 50  0001 C CNN
+F 2 "Connector_Molex:Molex_Mini-Fit_Sr_42819-22XX_1x02_P10.00mm_Vertical" H 11250 7350 50  0001 C CNN
 F 3 "~" H 11250 7350 50  0001 C CNN
 	1    11250 7350
@@
 F 0 "J11" H 12179 7342 50  0000 L CNN
 F 1 "MOTOR_2" H 12179 7251 50  0000 L CNN
-F 2 "Connector_Molex:Molex_Mini-Fit_Sr_42819-22XX_1x02_P10.00mm_Vertical_ThermalVias" H 12100 7350 50  0001 C CNN
+F 2 "Connector_Molex:Molex_Mini-Fit_Sr_42819-22XX_1x02_P10.00mm_Vertical" H 12100 7350 50  0001 C CNN
 F 3 "~" H 12100 7350 50  0001 C CNN
 	1    12100 7350
@@
 F 0 "J13" H 13029 7342 50  0000 L CNN
 F 1 "MOTOR_3" H 13029 7251 50  0000 L CNN
-F 2 "Connector_Molex:Molex_Mini-Fit_Sr_42819-22XX_1x02_P10.00mm_Vertical_ThermalVias" H 12950 7350 50  0001 C CNN
+F 2 "Connector_Molex:Molex_Mini-Fit_Sr_42819-22XX_1x02_P10.00mm_Vertical" H 12950 7350 50  0001 C CNN
 F 3 "~" H 12950 7350 50  0001 C CNN
 	1    12950 7350
@@
 F 0 "J15" H 13879 7342 50  0000 L CNN
 F 1 "MOTOR_4" H 13879 7251 50  0000 L CNN
-F 2 "Connector_Molex:Molex_Mini-Fit_Sr_42819-22XX_1x02_P10.00mm_Vertical_ThermalVias" H 13800 7350 50  0001 C CNN
+F 2 "Connector_Molex:Molex_Mini-Fit_Sr_42819-22XX_1x02_P10.00mm_Vertical" H 13800 7350 50  0001 C CNN
 F 3 "~" H 13800 7350 50  0001 C CNN
 	1    13800 7350
@@
 F 0 "J8" H 11329 8242 50  0000 L CNN
 F 1 "MOTOR_5" H 11329 8151 50  0000 L CNN
-F 2 "Connector_Molex:Molex_Mini-Fit_Sr_42819-22XX_1x02_P10.00mm_Vertical_ThermalVias" H 11250 8250 50  0001 C CNN
+F 2 "Connector_Molex:Molex_Mini-Fit_Sr_42819-22XX_1x02_P10.00mm_Vertical" H 11250 8250 50  0001 C CNN
 F 3 "~" H 11250 8250 50  0001 C CNN
 	1    11250 8250
@@
 F 0 "J12" H 12179 8242 50  0000 L CNN
 F 1 "MOTOR_6" H 12179 8151 50  0000 L CNN
-F 2 "Connector_Molex:Molex_Mini-Fit_Sr_42819-22XX_1x02_P10.00mm_Vertical_ThermalVias" H 12100 8250 50  0001 C CNN
+F 2 "Connector_Molex:Molex_Mini-Fit_Sr_42819-22XX_1x02_P10.00mm_Vertical" H 12100 8250 50  0001 C CNN
 F 3 "~" H 12100 8250 50  0001 C CNN
 	1    12100 8250
@@
 F 0 "J14" H 13029 8242 50  0000 L CNN
 F 1 "MOTOR_7" H 13029 8151 50  0000 L CNN
-F 2 "Connector_Molex:Molex_Mini-Fit_Sr_42819-22XX_1x02_P10.00mm_Vertical_ThermalVias" H 12950 8250 50  0001 C CNN
+F 2 "Connector_Molex:Molex_Mini-Fit_Sr_42819-22XX_1x02_P10.00mm_Vertical" H 12950 8250 50  0001 C CNN
 F 3 "~" H 12950 8250 50  0001 C CNN
 	1    12950 8250
@@
 F 0 "J16" H 13879 8242 50  0000 L CNN
 F 1 "MOTOR_8" H 13879 8151 50  0000 L CNN
-F 2 "Connector_Molex:Molex_Mini-Fit_Sr_42819-22XX_1x02_P10.00mm_Vertical_ThermalVias" H 13800 8250 50  0001 C CNN
+F 2 "Connector_Molex:Molex_Mini-Fit_Sr_42819-22XX_1x02_P10.00mm_Vertical" H 13800 8250 50  0001 C CNN
 F 3 "~" H 13800 8250 50  0001 C CNN
 	1    13800 8250
@@
 Text Notes 11900 8800 0    50   ~ 0
 check current rating on headers!
+Wire Wire Line
+	4800 9000 4800 8900
+$Comp
+L power:+48V #PWR0132
+U 1 1 5C795A90
+P 5200 8200
+F 0 "#PWR0132" H 5200 8050 50  0001 C CNN
+F 1 "+48V" H 5215 8373 50  0000 C CNN
+F 2 "" H 5200 8200 50  0001 C CNN
+F 3 "" H 5200 8200 50  0001 C CNN
+	1    5200 8200
+	1    0    0    -1
+$EndComp
+$Comp
+L Connector_Generic:Conn_01x02 J4
+U 1 1 5C795DE3
+P 5500 8300
+F 0 "J4" H 5580 8292 50  0000 L CNN
+F 1 "Switch_A" H 5580 8201 50  0000 L CNN
+F 2 "Connector_Molex:Molex_Nano-Fit_105309-xx02_1x02_P2.50mm_Vertical" H 5500 8300 50  0001 C CNN
+F 3 "~" H 5500 8300 50  0001 C CNN
+	1    5500 8300
+	1    0    0    -1
+$EndComp
+$Comp
+L Connector_Generic:Conn_01x02 J17
+U 1 1 5C795EB3
+P 5500 8500
+F 0 "J17" H 5580 8492 50  0000 L CNN
+F 1 "Switch_B" H 5580 8401 50  0000 L CNN
+F 2 "Connector_Molex:Molex_Nano-Fit_105309-xx02_1x02_P2.50mm_Vertical" H 5500 8500 50  0001 C CNN
+F 3 "~" H 5500 8500 50  0001 C CNN
+	1    5500 8500
+	1    0    0    -1
+$EndComp
+$Comp
+L Connector_Generic:Conn_01x02 J18
+U 1 1 5C795F5B
+P 5500 8700
+F 0 "J18" H 5580 8692 50  0000 L CNN
+F 1 "Switch_C" H 5580 8601 50  0000 L CNN
+F 2 "Connector_Molex:Molex_Nano-Fit_105309-xx02_1x02_P2.50mm_Vertical" H 5500 8700 50  0001 C CNN
+F 3 "~" H 5500 8700 50  0001 C CNN
+	1    5500 8700
+	1    0    0    -1
+$EndComp
+$Comp
+L Connector_Generic:Conn_01x02 J19
+U 1 1 5C795FF9
+P 5500 8900
+F 0 "J19" H 5580 8892 50  0000 L CNN
+F 1 "Switch_D" H 5580 8801 50  0000 L CNN
+F 2 "Connector_Molex:Molex_Nano-Fit_105309-xx02_1x02_P2.50mm_Vertical" H 5500 8900 50  0001 C CNN
+F 3 "~" H 5500 8900 50  0001 C CNN
+	1    5500 8900
+	1    0    0    -1
+$EndComp
+Wire Wire Line
+	5300 8400 5200 8400
+Wire Wire Line
+	5200 8400 5200 8200
+Wire Wire Line
+	5300 8600 5200 8600
+Wire Wire Line
+	5200 8600 5200 8400
+Connection ~ 5200 8400
+Wire Wire Line
+	5300 8800 5200 8800
+Wire Wire Line
+	5200 8800 5200 8600
+Connection ~ 5200 8600
+Wire Wire Line
+	5300 9000 5200 9000
+Wire Wire Line
+	5200 9000 5200 8800
+Connection ~ 5200 8800
+Wire Wire Line
+	5300 8900 4800 8900
+Wire Wire Line
+	5300 8700 3850 8700
+Wire Wire Line
+	3850 8700 3850 9000
+Wire Wire Line
+	5300 8500 2900 8500
+Wire Wire Line
+	2900 8500 2900 9000
+Wire Wire Line
+	5300 8300 1950 8300
+Wire Wire Line
+	1950 8300 1950 9000
+Text Notes 1300 4650 0    50   ~ 0
+DO NOT CONNECT 12V AND 48V SIMUTANIOUSLY!!!!
 $EndSCHEMATC

Commit message: assigned part number and footprint to transistors
Parts:
- Q1, Q2, Q3, Q4: footprint (none) -> Package_TO_SOT_SMD:TO-252-3_TabPin2; Digikey part number (none) -> BTS3046SDRATMA1CT-ND
Changed lines of the file:
@@
 F 0 "Q1" H 2055 9246 50  0000 L CNN
 F 1 "Q_NMOS_GDS" H 2055 9155 50  0000 L CNN
-F 2 "" H 2050 9300 50  0001 C CNN
+F 2 "Package_TO_SOT_SMD:TO-252-3_TabPin2" H 2050 9300 50  0001 C CNN
 F 3 "~" H 1850 9200 50  0001 C CNN
+F 4 "BTS3046SDRATMA1CT-ND" H 0   0   50  0001 C CNN "Digikey part number"
 	1    1850 9200
 	1    0    0    -1
@@
 F 0 "Q2" H 3005 9246 50  0000 L CNN
 F 1 "Q_NMOS_GDS" H 3005 9155 50  0000 L CNN
-F 2 "" H 3000 9300 50  0001 C CNN
+F 2 "Package_TO_SOT_SMD:TO-252-3_TabPin2" H 3000 9300 50  0001 C CNN
 F 3 "~" H 2800 9200 50  0001 C CNN
+F 4 "BTS3046SDRATMA1CT-ND" H 0   0   50  0001 C CNN "Digikey part number"
 	1    2800 9200
 	1    0    0    -1
@@
 F 0 "Q3" H 3955 9246 50  0000 L CNN
 F 1 "Q_NMOS_GDS" H 3955 9155 50  0000 L CNN
-F 2 "" H 3950 9300 50  0001 C CNN
+F 2 "Package_TO_SOT_SMD:TO-252-3_TabPin2" H 3950 9300 50  0001 C CNN
 F 3 "~" H 3750 9200 50  0001 C CNN
+F 4 "BTS3046SDRATMA1CT-ND" H 0   0   50  0001 C CNN "Digikey part number"
 	1    3750 9200
 	1    0    0    -1
@@
 F 0 "Q4" H 4905 9246 50  0000 L CNN
 F 1 "Q_NMOS_GDS" H 4905 9155 50  0000 L CNN
-F 2 "" H 4900 9300 50  0001 C CNN
+F 2 "Package_TO_SOT_SMD:TO-252-3_TabPin2" H 4900 9300 50  0001 C CNN
 F 3 "~" H 4700 9200 50  0001 C CNN
+F 4 "BTS3046SDRATMA1CT-ND" H 0   0   50  0001 C CNN "Digikey part number"
 	1    4700 9200
 	1    0    0    -1

Commit message: Added thermal vias to switches, just in case
Other:
- note added: "Add LED indicators"
Changed lines of the file:
@@
 Text Notes 1300 4650 0    50   ~ 0
 DO NOT CONNECT 12V AND 48V SIMUTANIOUSLY!!!!
+Text Notes 1500 9850 0    50   ~ 0
+Add LED indicators
 $EndSCHEMATC

Commit message: added leds for low side switches
Parts:
- added D4, D5, D6, D7: LED, LED_SMD:LED_0603_1608Metric_Pad1.05x0.95mm_HandSolder, symbol Device:LED
- added R12, R13, R14, R15: R_Small, Resistor_SMD:R_0603_1608Metric_Pad1.05x0.95mm_HandSolder, symbol Device:R_Small
Connections:
- wire segments 288 -> 304
Changed lines of the file:
@@
 Text Notes 1500 9850 0    50   ~ 0
 Add LED indicators
+$Comp
+L Device:LED D4
+U 1 1 5C5E06A0
+P 7250 9050
+F 0 "D4" H 7242 8795 50  0000 C CNN
+F 1 "LED" H 7242 8886 50  0000 C CNN
+F 2 "LED_SMD:LED_0603_1608Metric_Pad1.05x0.95mm_HandSolder" H 7250 9050 50  0001 C CNN
+F 3 "~" H 7250 9050 50  0001 C CNN
+	1    7250 9050
+	-1   0    0    1
+$EndComp
+$Comp
+L Device:LED D5
+U 1 1 5C5E0B13
+P 7250 9400
+F 0 "D5" H 7242 9145 50  0000 C CNN
+F 1 "LED" H 7242 9236 50  0000 C CNN
+F 2 "LED_SMD:LED_0603_1608Metric_Pad1.05x0.95mm_HandSolder" H 7250 9400 50  0001 C CNN
+F 3 "~" H 7250 9400 50  0001 C CNN
+	1    7250 9400
+	-1   0    0    1
+$EndComp
+$Comp
+L Device:LED D6
+U 1 1 5C5E0C35
+P 7250 9750
+F 0 "D6" H 7242 9495 50  0000 C CNN
+F 1 "LED" H 7242 9586 50  0000 C CNN
+F 2 "LED_SMD:LED_0603_1608Metric_Pad1.05x0.95mm_HandSolder" H 7250 9750 50  0001 C CNN
+F 3 "~" H 7250 9750 50  0001 C CNN
+	1    7250 9750
+	-1   0    0    1
+$EndComp
+$Comp
+L Device:LED D7
+U 1 1 5C5E1323
+P 7250 10100
+F 0 "D7" H 7242 9845 50  0000 C CNN
+F 1 "LED" H 7242 9936 50  0000 C CNN
+F 2 "LED_SMD:LED_0603_1608Metric_Pad1.05x0.95mm_HandSolder" H 7250 10100 50  0001 C CNN
+F 3 "~" H 7250 10100 50  0001 C CNN
+	1    7250 10100
+	-1   0    0    1
+$EndComp
+$Comp
+L Device:R_Small R12
+U 1 1 5C5E15B3
+P 6850 9050
+F 0 "R12" V 6654 9050 50  0000 C CNN
+F 1 "R_Small" V 6745 9050 50  0000 C CNN
+F 2 "Resistor_SMD:R_0603_1608Metric_Pad1.05x0.95mm_HandSolder" H 6850 9050 50  0001 C CNN
+F 3 "~" H 6850 9050 50  0001 C CNN
+	1    6850 9050
+	0    1    1    0
+$EndComp
+$Comp
+L Device:R_Small R13
+U 1 1 5C5E16A7
+P 6850 9400
+F 0 "R13" V 6654 9400 50  0000 C CNN
+F 1 "R_Small" V 6745 9400 50  0000 C CNN
+F 2 "Resistor_SMD:R_0603_1608Metric_Pad1.05x0.95mm_HandSolder" H 6850 9400 50  0001 C CNN
+F 3 "~" H 6850 9400 50  0001 C CNN
+	1    6850 9400
+	0    1    1    0
+$EndComp
+$Comp
+L Device:R_Small R14
+U 1 1 5C5E1792
+P 6850 9750
+F 0 "R14" V 6654 9750 50  0000 C CNN
+F 1 "R_Small" V 6745 9750 50  0000 C CNN
+F 2 "Resistor_SMD:R_0603_1608Metric_Pad1.05x0.95mm_HandSolder" H 6850 9750 50  0001 C CNN
+F 3 "~" H 6850 9750 50  0001 C CNN
+	1    6850 9750
+	0    1    1    0
+$EndComp
+$Comp
+L Device:R_Small R15
+U 1 1 5C5E1888
+P 6850 10100
+F 0 "R15" V 6654 10100 50  0000 C CNN
+F 1 "R_Small" V 6745 10100 50  0000 C CNN
+F 2 "Resistor_SMD:R_0603_1608Metric_Pad1.05x0.95mm_HandSolder" H 6850 10100 50  0001 C CNN
+F 3 "~" H 6850 10100 50  0001 C CNN
+	1    6850 10100
+	0    1    1    0
+$EndComp
+$Comp
+L power:GND #PWR0114
+U 1 1 5C5E1983
+P 7500 9100
+F 0 "#PWR0114" H 7500 8850 50  0001 C CNN
+F 1 "GND" H 7505 8927 50  0000 C CNN
+F 2 "" H 7500 9100 50  0001 C CNN
+F 3 "" H 7500 9100 50  0001 C CNN
+	1    7500 9100
+	1    0    0    -1
+$EndComp
+$Comp
+L power:GND #PWR0159
+U 1 1 5C5E1A25
+P 7500 9450
+F 0 "#PWR0159" H 7500 9200 50  0001 C CNN
+F 1 "GND" H 7505 9277 50  0000 C CNN
+F 2 "" H 7500 9450 50  0001 C CNN
+F 3 "" H 7500 9450 50  0001 C CNN
+	1    7500 9450
+	1    0    0    -1
+$EndComp
+$Comp
+L power:GND #PWR0160
+U 1 1 5C5E1AC7
+P 7500 9800
+F 0 "#PWR0160" H 7500 9550 50  0001 C CNN
+F 1 "GND" H 7505 9627 50  0000 C CNN
+F 2 "" H 7500 9800 50  0001 C CNN
+F 3 "" H 7500 9800 50  0001 C CNN
+	1    7500 9800
+	1    0    0    -1
+$EndComp
+$Comp
+L power:GND #PWR0161
+U 1 1 5C5E1B69
+P 7500 10150
+F 0 "#PWR0161" H 7500 9900 50  0001 C CNN
+F 1 "GND" H 7505 9977 50  0000 C CNN
+F 2 "" H 7500 10150 50  0001 C CNN
+F 3 "" H 7500 10150 50  0001 C CNN
+	1    7500 10150
+	1    0    0    -1
+$EndComp
+Text Label 6350 9050 0    50   ~ 0
+SWITCH_A
+Text Label 6350 9400 0    50   ~ 0
+SWITCH_B
+Text Label 6350 9750 0    50   ~ 0
+SWITCH_C
+Text Label 6350 10100 0    50   ~ 0
+SWITCH_D
+Wire Wire Line
+	7500 9100 7500 9050
+Wire Wire Line
+	7500 9050 7400 9050
+Wire Wire Line
+	7500 9450 7500 9400
+Wire Wire Line
+	7500 9400 7400 9400
+Wire Wire Line
+	7500 9800 7500 9750
+Wire Wire Line
+	7500 9750 7400 9750
+Wire Wire Line
+	7500 10150 7500 10100
+Wire Wire Line
+	7500 10100 7400 10100
+Wire Wire Line
+	7100 10100 6950 10100
+Wire Wire Line
+	7100 9750 6950 9750
+Wire Wire Line
+	7100 9400 6950 9400
+Wire Wire Line
+	7100 9050 6950 9050
+Wire Wire Line
+	6750 9050 6350 9050
+Wire Wire Line
+	6350 9400 6750 9400
+Wire Wire Line
+	6750 9750 6350 9750
+Wire Wire Line
+	6750 10100 6350 10100
 $EndSCHEMATC

Commit message: changed nano-fit footprint to have sort-of not intersecting pads
Parts:
- J17, J18, J19, J4: footprint Connector_Molex:Molex_Nano-Fit_105309-xx02_1x02_P2.50mm_Vertical -> footprints:Molex_Nano-Fit_105309-xx02_1x02_P2.50mm_Vertical_Oval_Pads
Changed lines of the file:
@@
 F 0 "J4" H 5580 8292 50  0000 L CNN
 F 1 "Switch_A" H 5580 8201 50  0000 L CNN
-F 2 "Connector_Molex:Molex_Nano-Fit_105309-xx02_1x02_P2.50mm_Vertical" H 5500 8300 50  0001 C CNN
+F 2 "footprints:Molex_Nano-Fit_105309-xx02_1x02_P2.50mm_Vertical_Oval_Pads" H 5500 8300 50  0001 C CNN
 F 3 "~" H 5500 8300 50  0001 C CNN
 	1    5500 8300
@@
 F 0 "J17" H 5580 8492 50  0000 L CNN
 F 1 "Switch_B" H 5580 8401 50  0000 L CNN
-F 2 "Connector_Molex:Molex_Nano-Fit_105309-xx02_1x02_P2.50mm_Vertical" H 5500 8500 50  0001 C CNN
+F 2 "footprints:Molex_Nano-Fit_105309-xx02_1x02_P2.50mm_Vertical_Oval_Pads" H 5500 8500 50  0001 C CNN
 F 3 "~" H 5500 8500 50  0001 C CNN
 	1    5500 8500
@@
 F 0 "J18" H 5580 8692 50  0000 L CNN
 F 1 "Switch_C" H 5580 8601 50  0000 L CNN
-F 2 "Connector_Molex:Molex_Nano-Fit_105309-xx02_1x02_P2.50mm_Vertical" H 5500 8700 50  0001 C CNN
+F 2 "footprints:Molex_Nano-Fit_105309-xx02_1x02_P2.50mm_Vertical_Oval_Pads" H 5500 8700 50  0001 C CNN
 F 3 "~" H 5500 8700 50  0001 C CNN
 	1    5500 8700
@@
 F 0 "J19" H 5580 8892 50  0000 L CNN
 F 1 "Switch_D" H 5580 8801 50  0000 L CNN
-F 2 "Connector_Molex:Molex_Nano-Fit_105309-xx02_1x02_P2.50mm_Vertical" H 5500 8900 50  0001 C CNN
+F 2 "footprints:Molex_Nano-Fit_105309-xx02_1x02_P2.50mm_Vertical_Oval_Pads" H 5500 8900 50  0001 C CNN
 F 3 "~" H 5500 8900 50  0001 C CNN
 	1    5500 8900
