File: electrical/control board power/control board power.sch (KiCad schematic (older format))
At the start: 64 parts, among them J10 48V_from_conversion, J11 MOTOR_2, J12 MOTOR_6, J13 MOTOR_3, J14 MOTOR_7, J15 MOTOR_4, J16 MOTOR_8, J17 Switch_B, J18 Switch_C, J19 Switch_D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

Commit message: Created symbol and footprint for other terminal strip
Parts:
- removed J11: MOTOR_2, Connector_Molex:Molex_Mini-Fit_Sr_42819-22XX_1x02_P10.00mm_Vertical, symbol Connector_Generic:Conn_01x02
- removed J12: MOTOR_6, Connector_Molex:Molex_Mini-Fit_Sr_42819-22XX_1x02_P10.00mm_Vertical, symbol Connector_Generic:Conn_01x02
- removed J13: MOTOR_3, Connector_Molex:Molex_Mini-Fit_Sr_42819-22XX_1x02_P10.00mm_Vertical, symbol Connector_Generic:Conn_01x02
- removed J14: MOTOR_7, Connector_Molex:Molex_Mini-Fit_Sr_42819-22XX_1x02_P10.00mm_Vertical, symbol Connector_Generic:Conn_01x02
- removed J15: MOTOR_4, Connector_Molex:Molex_Mini-Fit_Sr_42819-22XX_1x02_P10.00mm_Vertical, symbol Connector_Generic:Conn_01x02
- removed J16: MOTOR_8, Connector_Molex:Molex_Mini-Fit_Sr_42819-22XX_1x02_P10.00mm_Vertical, symbol Connector_Generic:Conn_01x02
- removed J7: MOTOR_1, Connector_Molex:Molex_Mini-Fit_Sr_42819-22XX_1x02_P10.00mm_Vertical, symbol Connector_Generic:Conn_01x02
- removed J8: MOTOR_5, Connector_Molex:Molex_Mini-Fit_Sr_42819-22XX_1x02_P10.00mm_Vertical, symbol Connector_Generic:Conn_01x02
- removed J9: 24V_from_conversion, Connector_Molex:Molex_Mini-Fit_Jr_5566-08A2_2x04_P4.20mm_Vertical, symbol Connector_Generic:Conn_02x04_Top_Bottom
Connections:
- wire segments 304 -> 253
Other:
- note removed: "No ground on this connector\nis intentional"
- note removed: "check current rating on headers!"

Commit message: replaced motor headers with mounting point for terminal block
Parts:
- added TB1: Curtis_2000, footprints:Curtis_2010, symbol custom_symbols:Curtis_2000
Changed lines of the file:
@@
 Wire Wire Line
 	6750 10100 6350 10100
+$Comp
+L custom_symbols:Curtis_2000 TB1
+U 1 1 5C643645
+P 9800 6700
+F 0 "TB1" H 9800 6815 50  0000 C CNN
+F 1 "Curtis_2000" H 9800 6724 50  0000 C CNN
+F 2 "footprints:Curtis_2010" H 9800 6700 50  0001 C CNN
+F 3 "" H 9800 6700 50  0001 C CNN
+	1    9800 6700
+	1    0    0    -1
+$EndComp
 $EndSCHEMATC
