File: electrical/control board power/control board power.sch (KiCad schematic (older format))
At the start: 56 parts, among them J10 48V_from_conversion, J17 Switch_B, J18 Switch_C, J19 Switch_D, J2 5V, J3 Barrel_Jack, J4 Switch_A, J5 Switch_Input, J6 Power_Connector, Q1 Q_NMOS_GDS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

Commit message: Stuff
Parts:
- added C15, C16, C17, C18: 22uF, Capacitor_SMD:C_1210_3225Metric_Pad1.42x2.65mm_HandSolder, symbol Device:C_Small
- added D8: LED, LED_SMD:LED_0603_1608Metric_Pad1.05x0.95mm_HandSolder, symbol Device:LED
- added J1: Conn_01x02, footprints:Molex_Nano-Fit_105309-xx02_1x02_P2.50mm_Vertical_Oval_Pads, symbol Connector_Generic:Conn_01x02
- added R16: R_Small, Resistor_SMD:R_0603_1608Metric_Pad1.05x0.95mm_HandSolder, symbol Device:R_Small
- added TB2: Curtis_2000, symbol custom_symbols:Curtis_2000
- C12, C13: footprint Capacitor_SMD:C_0603_1608Metric_Pad1.05x0.95mm_HandSolder -> Capacitor_SMD:C_1210_3225Metric_Pad1.42x2.65mm_HandSolder
Connections:
- wire segments 253 -> 274
Other:
- note added: "Consider breaking this up into more capacitors"
- note added: "Note: Stack terminal blocks"

Commit message: stuff
Parts:
- added C19, C20: 2.2uF, Capacitor_SMD:C_1210_3225Metric_Pad1.42x2.65mm_HandSolder, symbol Device:C_Small
- added C21, C22: 0.1uF, Capacitor_SMD:C_0805_2012Metric_Pad1.15x1.40mm_HandSolder, symbol Device:C_Small
- C3, C4: value 4.7uF -> 2.2uF; footprint Capacitor_SMD:C_0603_1608Metric_Pad1.05x0.95mm_HandSolder -> Capacitor_SMD:C_1210_3225Metric_Pad1.42x2.65mm_HandSolder
Connections:
- net labels removed: +12V
- wire segments 274 -> 295
Other:
- note removed: "Consider breaking this up into more capacitors"
Changed lines of the file:
@@
 NoConn ~ 5900 5500
-$Comp
-L power:GND #PWR0115
-U 1 1 5C97A8B2
-P 3650 5000
-F 0 "#PWR0115" H 3650 4750 50  0001 C CNN
-F 1 "GND" H 3655 4827 50  0000 C CNN
-F 2 "" H 3650 5000 50  0001 C CNN
-F 3 "" H 3650 5000 50  0001 C CNN
-	1    3650 5000
-	1    0    0    -1
-$EndComp
-$Comp
-L Device:C_Small C3
-U 1 1 5C97A8A9
-P 3650 4900
-F 0 "C3" H 3742 4946 50  0000 L CNN
-F 1 "4.7uF" H 3742 4855 50  0000 L CNN
-F 2 "Capacitor_SMD:C_0603_1608Metric_Pad1.05x0.95mm_HandSolder" H 3650 4900 50  0001 C CNN
-F 3 "~" H 3650 4900 50  0001 C CNN
-	1    3650 4900
-	1    0    0    -1
-$EndComp
-Connection ~ 3650 4800
-Wire Wire Line
-	4300 4800 3650 4800
-Wire Wire Line
-	3650 4800 3500 4800
-Wire Wire Line
-	3500 4800 3250 4800
-Connection ~ 3500 4800
-$Comp
-L power:+12V #PWR0116
-U 1 1 5C97A8A0
-P 3500 4800
-F 0 "#PWR0116" H 3500 4650 50  0001 C CNN
-F 1 "+12V" H 3515 4973 50  0000 C CNN
-F 2 "" H 3500 4800 50  0001 C CNN
-F 3 "" H 3500 4800 50  0001 C CNN
-	1    3500 4800
-	1    0    0    -1
-$EndComp
 $Comp
 L power:+48V #PWR0117
 U 1 1 5C97A89A
-P 3250 4800
-F 0 "#PWR0117" H 3250 4650 50  0001 C CNN
-F 1 "+48V" H 3265 4973 50  0000 C CNN
-F 2 "" H 3250 4800 50  0001 C CNN
-F 3 "" H 3250 4800 50  0001 C CNN
-	1    3250 4800
+P 3250 4750
+F 0 "#PWR0117" H 3250 4600 50  0001 C CNN
+F 1 "+48V" H 3265 4923 50  0000 C CNN
+F 2 "" H 3250 4750 50  0001 C CNN
+F 3 "" H 3250 4750 50  0001 C CNN
+	1    3250 4750
 	1    0    0    -1
 $EndComp
@@
 F 3 "~" H 7300 5150 50  0001 C CNN
 	1    7300 5150
-	1    0    0    -1
-$EndComp
-$Comp
-L power:GND #PWR0119
-U 1 1 5C9247EA
-P 3700 2200
-F 0 "#PWR0119" H 3700 1950 50  0001 C CNN
-F 1 "GND" H 3705 2027 50  0000 C CNN
-F 2 "" H 3700 2200 50  0001 C CNN
-F 3 "" H 3700 2200 50  0001 C CNN
-	1    3700 2200
-	1    0    0    -1
-$EndComp
-$Comp
-L Device:C_Small C4
-U 1 1 5C9246EF
-P 3700 2100
-F 0 "C4" H 3792 2146 50  0000 L CNN
-F 1 "4.7uF" H 3792 2055 50  0000 L CNN
-F 2 "Capacitor_SMD:C_0603_1608Metric_Pad1.05x0.95mm_HandSolder" H 3700 2100 50  0001 C CNN
-F 3 "~" H 3700 2100 50  0001 C CNN
-	1    3700 2100
-	1    0    0    -1
-$EndComp
-Connection ~ 3700 2000
-Wire Wire Line
-	4350 2000 3700 2000
-$Comp
-L power:+48V #PWR0121
-U 1 1 5C8FB0D4
-P 3300 2000
-F 0 "#PWR0121" H 3300 1850 50  0001 C CNN
-F 1 "+48V" H 3315 2173 50  0000 C CNN
-F 2 "" H 3300 2000 50  0001 C CNN
-F 3 "" H 3300 2000 50  0001 C CNN
-	1    3300 2000
 	1    0    0    -1
 $EndComp
@@
 	10650 5750 10650 5650
 Connection ~ 10650 5650
-Wire Wire Line
-	3300 2000 3700 2000
 $Comp
 L Device:LED D8
@@
 	2100 7150 2100 7050
 Connection ~ 2100 7050
-Text Notes 2850 2200 0    50   ~ 0
-Consider breaking this up into more capacitors
 $Comp
 L Device:C_Small C16
@@
 Connection ~ 8000 2400
 Connection ~ 7650 2400
+$Comp
+L Device:C_Small C3
+U 1 1 5C6F24E4
+P 2900 2200
+F 0 "C3" H 2992 2246 50  0000 L CNN
+F 1 "2.2uF" H 2992 2155 50  0000 L CNN
+F 2 "Capacitor_SMD:C_1210_3225Metric_Pad1.42x2.65mm_HandSolder" H 2900 2200 50  0001 C CNN
+F 3 "~" H 2900 2200 50  0001 C CNN
+	1    2900 2200
+	1    0    0    -1
+$EndComp
+$Comp
+L Device:C_Small C19
+U 1 1 5C6F27C4
+P 3300 2200
+F 0 "C19" H 3392 2246 50  0000 L CNN
+F 1 "2.2uF" H 3392 2155 50  0000 L CNN
+F 2 "Capacitor_SMD:C_1210_3225Metric_Pad1.42x2.65mm_HandSolder" H 3300 2200 50  0001 C CNN
+F 3 "~" H 3300 2200 50  0001 C CNN
+	1    3300 2200
+	1    0    0    -1
+$EndComp
+$Comp
+L Device:C_Small C21
+U 1 1 5C6F287A
+P 3700 2200
+F 0 "C21" H 3792 2246 50  0000 L CNN
+F 1 "0.1uF" H 3792 2155 50  0000 L CNN
+F 2 "Capacitor_SMD:C_0805_2012Metric_Pad1.15x1.40mm_HandSolder" H 3700 2200 50  0001 C CNN
+F 3 "~" H 3700 2200 50  0001 C CNN
+	1    3700 2200
+	1    0    0    -1
+$EndComp
+Wire Wire Line
+	2900 2000 2900 2100
+Wire Wire Line
+	2900 2000 3300 2000
+Wire Wire Line
+	3300 2100 3300 2000
+Connection ~ 3300 2000
+Wire Wire Line
+	3300 2000 3700 2000
+Wire Wire Line
+	3700 2100 3700 2000
+Connection ~ 3700 2000
+Wire Wire Line
+	3700 2000 4350 2000
+$Comp
+L power:+48V #PWR0115
+U 1 1 5C72C578
+P 2900 2000
+F 0 "#PWR0115" H 2900 1850 50  0001 C CNN
+F 1 "+48V" H 2915 2173 50  0000 C CNN
+F 2 "" H 2900 2000 50  0001 C CNN
+F 3 "" H 2900 2000 50  0001 C CNN
+	1    2900 2000
+	1    0    0    -1
+$EndComp
+Connection ~ 2900 2000
+$Comp
+L power:GND #PWR0116
+U 1 1 5C72C625
+P 3300 2400
+F 0 "#PWR0116" H 3300 2150 50  0001 C CNN
+F 1 "GND" H 3305 2227 50  0000 C CNN
+F 2 "" H 3300 2400 50  0001 C CNN
+F 3 "" H 3300 2400 50  0001 C CNN
+	1    3300 2400
+	1    0    0    -1
+$EndComp
+Wire Wire Line
+	2900 2300 2900 2350
+Wire Wire Line
+	2900 2350 3300 2350
+Wire Wire Line
+	3700 2350 3700 2300
+Wire Wire Line
+	3300 2300 3300 2350
+Connection ~ 3300 2350
+Wire Wire Line
+	3300 2350 3700 2350
+Wire Wire Line
+	3300 2400 3300 2350
+$Comp
+L Device:C_Small C4
+U 1 1 5C77D5F8
+P 3050 5050
+F 0 "C4" H 3142 5096 50  0000 L CNN
+F 1 "2.2uF" H 3142 5005 50  0000 L CNN
+F 2 "Capacitor_SMD:C_1210_3225Metric_Pad1.42x2.65mm_HandSolder" H 3050 5050 50  0001 C CNN
+F 3 "~" H 3050 5050 50  0001 C CNN
+	1    3050 5050
+	1    0    0    -1
+$EndComp
+$Comp
+L Device:C_Small C20
+U 1 1 5C77D5FE
+P 3450 5050
+F 0 "C20" H 3542 5096 50  0000 L CNN
+F 1 "2.2uF" H 3542 5005 50  0000 L CNN
+F 2 "Capacitor_SMD:C_1210_3225Metric_Pad1.42x2.65mm_HandSolder" H 3450 5050 50  0001 C CNN
+F 3 "~" H 3450 5050 50  0001 C CNN
+	1    3450 5050
+	1    0    0    -1
+$EndComp
+$Comp
+L Device:C_Small C22
+U 1 1 5C77D604
+P 3850 5050
+F 0 "C22" H 3942 5096 50  0000 L CNN
+F 1 "0.1uF" H 3942 5005 50  0000 L CNN
+F 2 "Capacitor_SMD:C_0805_2012Metric_Pad1.15x1.40mm_HandSolder" H 3850 5050 50  0001 C CNN
+F 3 "~" H 3850 5050 50  0001 C CNN
+	1    3850 5050
+	1    0    0    -1
+$EndComp
+$Comp
+L power:GND #PWR0119
+U 1 1 5C77D619
+P 3450 5250
+F 0 "#PWR0119" H 3450 5000 50  0001 C CNN
+F 1 "GND" H 3455 5077 50  0000 C CNN
+F 2 "" H 3450 5250 50  0001 C CNN
+F 3 "" H 3450 5250 50  0001 C CNN
+	1    3450 5250
+	1    0    0    -1
+$EndComp
+Wire Wire Line
+	3050 5150 3050 5200
+Wire Wire Line
+	3050 5200 3450 5200
+Wire Wire Line
+	3850 5200 3850 5150
+Wire Wire Line
+	3450 5150 3450 5200
+Connection ~ 3450 5200
+Wire Wire Line
+	3450 5200 3850 5200
+Wire Wire Line
+	3450 5250 3450 5200
+Wire Wire Line
+	3250 4800 3450 4800
+Wire Wire Line
+	3250 4750 3250 4800
+Wire Wire Line
+	3050 4800 3250 4800
+Wire Wire Line
+	3050 4800 3050 4950
+Connection ~ 3250 4800
+Wire Wire Line
+	3450 4800 3450 4950
+Connection ~ 3450 4800
+Wire Wire Line
+	3450 4800 3850 4800
+Wire Wire Line
+	3850 4800 3850 4950
+Connection ~ 3850 4800
+Wire Wire Line
+	3850 4800 4300 4800
 $EndSCHEMATC

Commit message: Found some parts
Parts:
- C1, C2: Digikey part number (none) -> 490-7198-1-ND
- C10: Digikey part number (none) -> 732-8003-1-ND
- C11: Digikey part number (none) -> 732-7947-1-ND
- C12, C13, C15, C16, C17, C18: Digikey part number (none) -> 1276-1855-1-ND
- C19, C20, C3, C4: Digikey part number (none) -> 445-4497-1-ND
- C21, C22: Digikey part number (none) -> 732-12244-1-ND
- C5, C7: Digikey part number (none) -> 478-5010-1-ND
- C6, C8: Digikey part number (none) -> 399-1100-1-ND
- C9: Digikey part number (none) -> 732-7760-1-ND
- R16, R3: footprint Resistor_SMD:R_0603_1608Metric_Pad1.05x0.95mm_HandSolder -> Resistor_SMD:R_1206_3216Metric_Pad1.42x1.75mm_HandSolder
Changed lines of the file:
@@
 F 0 "R3" V 1596 6700 50  0000 C CNN
 F 1 "R_Small" V 1505 6700 50  0000 C CNN
-F 2 "Resistor_SMD:R_0603_1608Metric_Pad1.05x0.95mm_HandSolder" H 1400 6700 50  0001 C CNN
+F 2 "Resistor_SMD:R_1206_3216Metric_Pad1.42x1.75mm_HandSolder" H 1400 6700 50  0001 C CNN
 F 3 "~" H 1400 6700 50  0001 C CNN
 	1    1400 6700
@@
 F 2 "Capacitor_SMD:C_0603_1608Metric_Pad1.05x0.95mm_HandSolder" H 2650 4150 50  0001 C CNN
 F 3 "~" H 2650 4150 50  0001 C CNN
+F 4 "490-7198-1-ND" H 0   0   50  0001 C CNN "Digikey part number"
 	1    2650 4150
 	1    0    0    -1
@@
 F 2 "Capacitor_SMD:C_0603_1608Metric_Pad1.05x0.95mm_HandSolder" H 1600 4150 50  0001 C CNN
 F 3 "~" H 1600 4150 50  0001 C CNN
+F 4 "490-7198-1-ND" H 0   0   50  0001 C CNN "Digikey part number"
 	1    1600 4150
 	1    0    0    -1
@@
 F 2 "Capacitor_SMD:C_1210_3225Metric_Pad1.42x2.65mm_HandSolder" H 7300 5150 50  0001 C CNN
 F 3 "~" H 7300 5150 50  0001 C CNN
+F 4 "1276-1855-1-ND" H 0   0   50  0001 C CNN "Digikey part number"
 	1    7300 5150
 	1    0    0    -1
@@
 F 2 "Capacitor_SMD:C_1210_3225Metric_Pad1.42x2.65mm_HandSolder" H 7650 2300 50  0001 C CNN
 F 3 "~" H 7650 2300 50  0001 C CNN
+F 4 "1276-1855-1-ND" H 0   0   50  0001 C CNN "Digikey part number"
 	1    7650 2300
 	1    0    0    -1
@@
 F 2 "Capacitor_SMD:C_0603_1608Metric_Pad1.05x0.95mm_HandSolder" H 6300 2100 50  0001 C CNN
 F 3 "~" H 6300 2100 50  0001 C CNN
+F 4 "399-1100-1-ND" H 0   0   50  0001 C CNN "Digikey part number"
 	1    6300 2100
 	1    0    0    -1
@@
 F 2 "Capacitor_SMD:C_0603_1608Metric_Pad1.05x0.95mm_HandSolder" H 6600 3250 50  0001 C CNN
 F 3 "~" H 6600 3250 50  0001 C CNN
+F 4 "732-7947-1-ND" H 0   0   50  0001 C CNN "Digikey part number"
 	1    6600 3250
 	0    1    1    0
@@
 F 2 "Capacitor_SMD:C_0603_1608Metric_Pad1.05x0.95mm_HandSolder" H 6600 2900 50  0001 C CNN
 F 3 "~" H 6600 2900 50  0001 C CNN
+F 4 "732-8003-1-ND " H 0   0   50  0001 C CNN "Digikey part number"
 	1    6600 2900
 	0    1    1    0
@@
 F 2 "Capacitor_SMD:C_0603_1608Metric_Pad1.05x0.95mm_HandSolder" H 6150 3200 50  0001 C CNN
 F 3 "~" H 6150 3200 50  0001 C CNN
+F 4 "478-5010-1-ND" H 0   0   50  0001 C CNN "Digikey part number"
 	1    6150 3200
 	1    0    0    -1
@@
 F 2 "Capacitor_SMD:C_0603_1608Metric_Pad1.05x0.95mm_HandSolder" H 6050 4900 50  0001 C CNN
 F 3 "~" H 6050 4900 50  0001 C CNN
+F 4 "399-1100-1-ND" H 0   0   50  0001 C CNN "Digikey part number"
 	1    6050 4900
 	1    0    0    -1
@@
 F 2 "Capacitor_SMD:C_0603_1608Metric_Pad1.05x0.95mm_HandSolder" H 6350 6100 50  0001 C CNN
 F 3 "~" H 6350 6100 50  0001 C CNN
+F 4 "732-7760-1-ND" H 0   0   50  0001 C CNN "Digikey part number"
 	1    6350 6100
 	1    0    0    -1
@@
 F 2 "Capacitor_SMD:C_0603_1608Metric_Pad1.05x0.95mm_HandSolder" H 6000 6100 50  0001 C CNN
 F 3 "~" H 6000 6100 50  0001 C CNN
+F 4 "478-5010-1-ND" H 0   0   50  0001 C CNN "Digikey part number"
 	1    6000 6100
 	1    0    0    -1
@@
 F 0 "R16" V 1596 7050 50  0000 C CNN
 F 1 "R_Small" V 1505 7050 50  0000 C CNN
-F 2 "Resistor_SMD:R_0603_1608Metric_Pad1.05x0.95mm_HandSolder" H 1400 7050 50  0001 C CNN
+F 2 "Resistor_SMD:R_1206_3216Metric_Pad1.42x1.75mm_HandSolder" H 1400 7050 50  0001 C CNN
 F 3 "~" H 1400 7050 50  0001 C CNN
 	1    1400 7050
@@
 F 2 "Capacitor_SMD:C_1210_3225Metric_Pad1.42x2.65mm_HandSolder" H 8000 2300 50  0001 C CNN
 F 3 "~" H 8000 2300 50  0001 C CNN
+F 4 "1276-1855-1-ND" H 0   0   50  0001 C CNN "Digikey part number"
 	1    8000 2300
 	1    0    0    -1
@@
 F 2 "Capacitor_SMD:C_1210_3225Metric_Pad1.42x2.65mm_HandSolder" H 8350 2300 50  0001 C CNN
 F 3 "~" H 8350 2300 50  0001 C CNN
+F 4 "1276-1855-1-ND" H 0   0   50  0001 C CNN "Digikey part number"
 	1    8350 2300
 	1    0    0    -1
@@
 F 2 "Capacitor_SMD:C_1210_3225Metric_Pad1.42x2.65mm_HandSolder" H 7650 5150 50  0001 C CNN
 F 3 "~" H 7650 5150 50  0001 C CNN
+F 4 "1276-1855-1-ND" H 0   0   50  0001 C CNN "Digikey part number"
 	1    7650 5150
 	1    0    0    -1
@@
 F 2 "Capacitor_SMD:C_1210_3225Metric_Pad1.42x2.65mm_HandSolder" H 8000 5150 50  0001 C CNN
 F 3 "~" H 8000 5150 50  0001 C CNN
+F 4 "1276-1855-1-ND" H 0   0   50  0001 C CNN "Digikey part number"
 	1    8000 5150
 	1    0    0    -1
@@
 F 2 "Capacitor_SMD:C_1210_3225Metric_Pad1.42x2.65mm_HandSolder" H 2900 2200 50  0001 C CNN
 F 3 "~" H 2900 2200 50  0001 C CNN
+F 4 "445-4497-1-ND" H 0   0   50  0001 C CNN "Digikey part number"
 	1    2900 2200
 	1    0    0    -1
@@
 F 2 "Capacitor_SMD:C_1210_3225Metric_Pad1.42x2.65mm_HandSolder" H 3300 2200 50  0001 C CNN
 F 3 "~" H 3300 2200 50  0001 C CNN
+F 4 "445-4497-1-ND" H 0   0   50  0001 C CNN "Digikey part number"
 	1    3300 2200
 	1    0    0    -1
@@
 F 2 "Capacitor_SMD:C_0805_2012Metric_Pad1.15x1.40mm_HandSolder" H 3700 2200 50  0001 C CNN
 F 3 "~" H 3700 2200 50  0001 C CNN
+F 4 "732-12244-1-ND" H 0   0   50  0001 C CNN "Digikey part number"
 	1    3700 2200
 	1    0    0    -1
@@
 F 2 "Capacitor_SMD:C_1210_3225Metric_Pad1.42x2.65mm_HandSolder" H 3050 5050 50  0001 C CNN
 F 3 "~" H 3050 5050 50  0001 C CNN
+F 4 "445-4497-1-ND" H 0   0   50  0001 C CNN "Digikey part number"
 	1    3050 5050
 	1    0    0    -1
@@
 F 2 "Capacitor_SMD:C_1210_3225Metric_Pad1.42x2.65mm_HandSolder" H 3450 5050 50  0001 C CNN
 F 3 "~" H 3450 5050 50  0001 C CNN
+F 4 "445-4497-1-ND" H 0   0   50  0001 C CNN "Digikey part number"
 	1    3450 5050
 	1    0    0    -1
@@
 F 2 "Capacitor_SMD:C_0805_2012Metric_Pad1.15x1.40mm_HandSolder" H 3850 5050 50  0001 C CNN
 F 3 "~" H 3850 5050 50  0001 C CNN
+F 4 "732-12244-1-ND" H 0   0   50  0001 C CNN "Digikey part number"
 	1    3850 5050
 	1    0    0    -1

Commit message: Making the low side switches beefier
Parts:
- added C23, C24, C25, C26: 10uF, Capacitor_SMD:C_1210_3225Metric_Pad1.42x2.65mm_HandSolder, symbol Device:C_Small
- J17, J18, J19, J4: footprint footprints:Molex_Nano-Fit_105309-xx02_1x02_P2.50mm_Vertical_Oval_Pads -> Connector_Molex:Molex_Mini-Fit_Jr_5566-02A_2x01_P4.20mm_Vertical
Connections:
- wire segments 295 -> 305
Other:
- note added: "Consider adding ability to switch\nbetween 24 and 48 V"
- note removed: "Add LED indicators"
Changed lines of the file:
@@
 Connection ~ 4400 9750
-Wire Wire Line
-	4400 9750 4800 9750
 Wire Wire Line
 	3450 9500 3450 9750
@@
 Wire Wire Line
 	1500 9500 1500 9750
-Wire Wire Line
-	1500 9750 1950 9750
 Connection ~ 1950 9750
 $Comp
@@
 F 0 "J4" H 5580 8292 50  0000 L CNN
 F 1 "Switch_A" H 5580 8201 50  0000 L CNN
-F 2 "footprints:Molex_Nano-Fit_105309-xx02_1x02_P2.50mm_Vertical_Oval_Pads" H 5500 8300 50  0001 C CNN
+F 2 "Connector_Molex:Molex_Mini-Fit_Jr_5566-02A_2x01_P4.20mm_Vertical" H 5500 8300 50  0001 C CNN
 F 3 "~" H 5500 8300 50  0001 C CNN
 	1    5500 8300
@@
 F 0 "J17" H 5580 8492 50  0000 L CNN
 F 1 "Switch_B" H 5580 8401 50  0000 L CNN
-F 2 "footprints:Molex_Nano-Fit_105309-xx02_1x02_P2.50mm_Vertical_Oval_Pads" H 5500 8500 50  0001 C CNN
+F 2 "Connector_Molex:Molex_Mini-Fit_Jr_5566-02A_2x01_P4.20mm_Vertical" H 5500 8500 50  0001 C CNN
 F 3 "~" H 5500 8500 50  0001 C CNN
 	1    5500 8500
@@
 F 0 "J18" H 5580 8692 50  0000 L CNN
 F 1 "Switch_C" H 5580 8601 50  0000 L CNN
-F 2 "footprints:Molex_Nano-Fit_105309-xx02_1x02_P2.50mm_Vertical_Oval_Pads" H 5500 8700 50  0001 C CNN
+F 2 "Connector_Molex:Molex_Mini-Fit_Jr_5566-02A_2x01_P4.20mm_Vertical" H 5500 8700 50  0001 C CNN
 F 3 "~" H 5500 8700 50  0001 C CNN
 	1    5500 8700
@@
 F 0 "J19" H 5580 8892 50  0000 L CNN
 F 1 "Switch_D" H 5580 8801 50  0000 L CNN
-F 2 "footprints:Molex_Nano-Fit_105309-xx02_1x02_P2.50mm_Vertical_Oval_Pads" H 5500 8900 50  0001 C CNN
+F 2 "Connector_Molex:Molex_Mini-Fit_Jr_5566-02A_2x01_P4.20mm_Vertical" H 5500 8900 50  0001 C CNN
 F 3 "~" H 5500 8900 50  0001 C CNN
 	1    5500 8900
@@
 Text Notes 1300 4650 0    50   ~ 0
 DO NOT CONNECT 12V AND 48V SIMUTANIOUSLY!!!!
-Text Notes 1500 9850 0    50   ~ 0
-Add LED indicators
 $Comp
 L Device:LED D4
@@
 Wire Wire Line
 	3850 4800 4300 4800
+$Comp
+L Device:C_Small C23
+U 1 1 5C82C7FF
+P 1950 9850
+F 0 "C23" H 2042 9896 50  0000 L CNN
+F 1 "10uF" H 2042 9805 50  0000 L CNN
+F 2 "Capacitor_SMD:C_1210_3225Metric_Pad1.42x2.65mm_HandSolder" H 1950 9850 50  0001 C CNN
+F 3 "~" H 1950 9850 50  0001 C CNN
+	1    1950 9850
+	1    0    0    -1
+$EndComp
+$Comp
+L Device:C_Small C26
+U 1 1 5C82CEB4
+P 4400 9850
+F 0 "C26" H 4492 9896 50  0000 L CNN
+F 1 "10uF" H 4492 9805 50  0000 L CNN
+F 2 "Capacitor_SMD:C_1210_3225Metric_Pad1.42x2.65mm_HandSolder" H 4400 9850 50  0001 C CNN
+F 3 "~" H 4400 9850 50  0001 C CNN
+	1    4400 9850
+	1    0    0    -1
+$EndComp
+$Comp
+L power:+48V #PWR0121
+U 1 1 5C82D014
+P 4750 9950
+F 0 "#PWR0121" H 4750 9800 50  0001 C CNN
+F 1 "+48V" H 4765 10123 50  0000 C CNN
+F 2 "" H 4750 9950 50  0001 C CNN
+F 3 "" H 4750 9950 50  0001 C CNN
+	1    4750 9950
+	1    0    0    -1
+$EndComp
+Wire Wire Line
+	4400 9950 4400 10000
+Wire Wire Line
+	4400 10000 4750 10000
+Wire Wire Line
+	4750 10000 4750 9950
+Text Notes 3300 10350 0    50   ~ 0
+Consider adding ability to switch\nbetween 24 and 48 V
+$Comp
+L power:+48V #PWR0141
+U 1 1 5C844D20
+P 1550 9950
+F 0 "#PWR0141" H 1550 9800 50  0001 C CNN
+F 1 "+48V" H 1565 10123 50  0000 C CNN
+F 2 "" H 1550 9950 50  0001 C CNN
+F 3 "" H 1550 9950 50  0001 C CNN
+	1    1550 9950
+	1    0    0    -1
+$EndComp
+Wire Wire Line
+	1950 9950 1950 10050
+Wire Wire Line
+	1950 10050 1550 10050
+Wire Wire Line
+	1550 10050 1550 9950
+$Comp
+L Device:C_Small C24
+U 1 1 5C85E18C
+P 2900 9850
+F 0 "C24" H 2992 9896 50  0000 L CNN
+F 1 "10uF" H 2992 9805 50  0000 L CNN
+F 2 "Capacitor_SMD:C_1210_3225Metric_Pad1.42x2.65mm_HandSolder" H 2900 9850 50  0001 C CNN
+F 3 "~" H 2900 9850 50  0001 C CNN
+	1    2900 9850
+	1    0    0    -1
+$EndComp
+$Comp
+L Device:C_Small C25
+U 1 1 5C88F44D
+P 3850 9850
+F 0 "C25" H 3942 9896 50  0000 L CNN
+F 1 "10uF" H 3942 9805 50  0000 L CNN
+F 2 "Capacitor_SMD:C_1210_3225Metric_Pad1.42x2.65mm_HandSolder" H 3850 9850 50  0001 C CNN
+F 3 "~" H 3850 9850 50  0001 C CNN
+	1    3850 9850
+	1    0    0    -1
+$EndComp
+Wire Wire Line
+	4400 9750 4800 9750
+Wire Wire Line
+	1500 9750 1950 9750
+Wire Wire Line
+	2900 9950 2900 10050
+Wire Wire Line
+	2900 10050 1950 10050
+Connection ~ 1950 10050
+Wire Wire Line
+	3850 9950 3850 10000
+Wire Wire Line
+	3850 10000 4400 10000
+Connection ~ 4400 10000
 $EndSCHEMATC
