File: electrical/control board power/control board power.sch (KiCad schematic (older format))
At the start: 72 parts, among them J1 Conn_01x02, J10 48V_from_conversion, J17 Switch_B, J18 Switch_C, J19 Switch_D, J2 5V, J3 Barrel_Jack, J4 Switch_A, J5 Switch_Input, J6 Power_Connector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

Commit message: stuff
Parts:
- added D10, D11, D12, D9: D_Small, Diode_SMD:D_SMC_Handsoldering, symbol Device:D_Small
- Q1, Q2, Q3, Q4: footprint Package_TO_SOT_SMD:TO-252-3_TabPin2 -> footprints:TO-252-3_2_Pin
Connections:
- wire segments 305 -> 309
Changed lines of the file:
@@
 F 0 "Q1" H 2055 9246 50  0000 L CNN
 F 1 "Q_NMOS_GDS" H 2055 9155 50  0000 L CNN
-F 2 "Package_TO_SOT_SMD:TO-252-3_TabPin2" H 2050 9300 50  0001 C CNN
+F 2 "footprints:TO-252-3_2_Pin" H 2050 9300 50  0001 C CNN
 F 3 "~" H 1850 9200 50  0001 C CNN
 F 4 "BTS3046SDRATMA1CT-ND" H 0   0   50  0001 C CNN "Digikey part number"
@@
 F 0 "Q2" H 3005 9246 50  0000 L CNN
 F 1 "Q_NMOS_GDS" H 3005 9155 50  0000 L CNN
-F 2 "Package_TO_SOT_SMD:TO-252-3_TabPin2" H 3000 9300 50  0001 C CNN
+F 2 "footprints:TO-252-3_2_Pin" H 3000 9300 50  0001 C CNN
 F 3 "~" H 2800 9200 50  0001 C CNN
 F 4 "BTS3046SDRATMA1CT-ND" H 0   0   50  0001 C CNN "Digikey part number"
@@
 F 0 "Q3" H 3955 9246 50  0000 L CNN
 F 1 "Q_NMOS_GDS" H 3955 9155 50  0000 L CNN
-F 2 "Package_TO_SOT_SMD:TO-252-3_TabPin2" H 3950 9300 50  0001 C CNN
+F 2 "footprints:TO-252-3_2_Pin" H 3950 9300 50  0001 C CNN
 F 3 "~" H 3750 9200 50  0001 C CNN
 F 4 "BTS3046SDRATMA1CT-ND" H 0   0   50  0001 C CNN "Digikey part number"
@@
 F 0 "Q4" H 4905 9246 50  0000 L CNN
 F 1 "Q_NMOS_GDS" H 4905 9155 50  0000 L CNN
-F 2 "Package_TO_SOT_SMD:TO-252-3_TabPin2" H 4900 9300 50  0001 C CNN
+F 2 "footprints:TO-252-3_2_Pin" H 4900 9300 50  0001 C CNN
 F 3 "~" H 4700 9200 50  0001 C CNN
 F 4 "BTS3046SDRATMA1CT-ND" H 0   0   50  0001 C CNN "Digikey part number"
@@
 	3850 10000 4400 10000
 Connection ~ 4400 10000
+$Comp
+L Device:D_Small D12
+U 1 1 5C8F42D5
+P 4800 8050
+F 0 "D12" V 4754 8118 50  0000 L CNN
+F 1 "D_Small" V 4845 8118 50  0000 L CNN
+F 2 "Diode_SMD:D_SMC_Handsoldering" V 4800 8050 50  0001 C CNN
+F 3 "~" V 4800 8050 50  0001 C CNN
+F 4 "SMCJ150CALFCT-ND" H 0   0   50  0001 C CNN "Digikey part number"
+	1    4800 8050
+	0    1    1    0
+$EndComp
+$Comp
+L Device:D_Small D11
+U 1 1 5C8F48E3
+P 3850 8050
+F 0 "D11" V 3804 8118 50  0000 L CNN
+F 1 "D_Small" V 3895 8118 50  0000 L CNN
+F 2 "Diode_SMD:D_SMC_Handsoldering" V 3850 8050 50  0001 C CNN
+F 3 "~" V 3850 8050 50  0001 C CNN
+F 4 "SMCJ150CALFCT-ND" H 0   0   50  0001 C CNN "Digikey part number"
+	1    3850 8050
+	0    1    1    0
+$EndComp
+$Comp
+L Device:D_Small D10
+U 1 1 5C8F5150
+P 2900 8050
+F 0 "D10" V 2854 8118 50  0000 L CNN
+F 1 "D_Small" V 2945 8118 50  0000 L CNN
+F 2 "Diode_SMD:D_SMC_Handsoldering" V 2900 8050 50  0001 C CNN
+F 3 "~" V 2900 8050 50  0001 C CNN
+F 4 "SMCJ150CALFCT-ND" H 0   0   50  0001 C CNN "Digikey part number"
+	1    2900 8050
+	0    1    1    0
+$EndComp
+$Comp
+L Device:D_Small D9
+U 1 1 5C8F5280
+P 1950 8050
+F 0 "D9" V 1904 8118 50  0000 L CNN
+F 1 "D_Small" V 1995 8118 50  0000 L CNN
+F 2 "Diode_SMD:D_SMC_Handsoldering" V 1950 8050 50  0001 C CNN
+F 3 "~" V 1950 8050 50  0001 C CNN
+F 4 "SMCJ150CALFCT-ND" H 0   0   50  0001 C CNN "Digikey part number"
+	1    1950 8050
+	0    1    1    0
+$EndComp
+Wire Wire Line
+	1950 8150 1950 8300
+Connection ~ 1950 8300
+Wire Wire Line
+	2900 8150 2900 8500
+Connection ~ 2900 8500
+Wire Wire Line
+	3850 8150 3850 8700
+Connection ~ 3850 8700
+Wire Wire Line
+	4800 8150 4800 8900
+Connection ~ 4800 8900
+$Comp
+L power:+48V #PWR04
+U 1 1 5C959928
+P 4800 7950
+F 0 "#PWR04" H 4800 7800 50  0001 C CNN
+F 1 "+48V" H 4815 8123 50  0000 C CNN
+F 2 "" H 4800 7950 50  0001 C CNN
+F 3 "" H 4800 7950 50  0001 C CNN
+	1    4800 7950
+	1    0    0    -1
+$EndComp
+$Comp
+L power:+48V #PWR03
+U 1 1 5C9599E2
+P 3850 7950
+F 0 "#PWR03" H 3850 7800 50  0001 C CNN
+F 1 "+48V" H 3865 8123 50  0000 C CNN
+F 2 "" H 3850 7950 50  0001 C CNN
+F 3 "" H 3850 7950 50  0001 C CNN
+	1    3850 7950
+	1    0    0    -1
+$EndComp
+$Comp
+L power:+48V #PWR02
+U 1 1 5C959A9C
+P 2900 7950
+F 0 "#PWR02" H 2900 7800 50  0001 C CNN
+F 1 "+48V" H 2915 8123 50  0000 C CNN
+F 2 "" H 2900 7950 50  0001 C CNN
+F 3 "" H 2900 7950 50  0001 C CNN
+	1    2900 7950
+	1    0    0    -1
+$EndComp
+$Comp
+L power:+48V #PWR01
+U 1 1 5C95A1DE
+P 1950 7950
+F 0 "#PWR01" H 1950 7800 50  0001 C CNN
+F 1 "+48V" H 1965 8123 50  0000 C CNN
+F 2 "" H 1950 7950 50  0001 C CNN
+F 3 "" H 1950 7950 50  0001 C CNN
+	1    1950 7950
+	1    0    0    -1
+$EndComp
 $EndSCHEMATC

Commit message: Added flyback diodes on low side switches
Parts:
- D10, D11, D12, D9: footprint Diode_SMD:D_SMC_Handsoldering -> footprints:D_SMC_Handsoldering_Diode_Mark
Changed lines of the file:
@@
 F 0 "D12" V 4754 8118 50  0000 L CNN
 F 1 "D_Small" V 4845 8118 50  0000 L CNN
-F 2 "Diode_SMD:D_SMC_Handsoldering" V 4800 8050 50  0001 C CNN
+F 2 "footprints:D_SMC_Handsoldering_Diode_Mark" V 4800 8050 50  0001 C CNN
 F 3 "~" V 4800 8050 50  0001 C CNN
 F 4 "SMCJ150CALFCT-ND" H 0   0   50  0001 C CNN "Digikey part number"
@@
 F 0 "D11" V 3804 8118 50  0000 L CNN
 F 1 "D_Small" V 3895 8118 50  0000 L CNN
-F 2 "Diode_SMD:D_SMC_Handsoldering" V 3850 8050 50  0001 C CNN
+F 2 "footprints:D_SMC_Handsoldering_Diode_Mark" V 3850 8050 50  0001 C CNN
 F 3 "~" V 3850 8050 50  0001 C CNN
 F 4 "SMCJ150CALFCT-ND" H 0   0   50  0001 C CNN "Digikey part number"
@@
 F 0 "D10" V 2854 8118 50  0000 L CNN
 F 1 "D_Small" V 2945 8118 50  0000 L CNN
-F 2 "Diode_SMD:D_SMC_Handsoldering" V 2900 8050 50  0001 C CNN
+F 2 "footprints:D_SMC_Handsoldering_Diode_Mark" V 2900 8050 50  0001 C CNN
 F 3 "~" V 2900 8050 50  0001 C CNN
 F 4 "SMCJ150CALFCT-ND" H 0   0   50  0001 C CNN "Digikey part number"
@@
 F 0 "D9" V 1904 8118 50  0000 L CNN
 F 1 "D_Small" V 1995 8118 50  0000 L CNN
-F 2 "Diode_SMD:D_SMC_Handsoldering" V 1950 8050 50  0001 C CNN
+F 2 "footprints:D_SMC_Handsoldering_Diode_Mark" V 1950 8050 50  0001 C CNN
 F 3 "~" V 1950 8050 50  0001 C CNN
 F 4 "SMCJ150CALFCT-ND" H 0   0   50  0001 C CNN "Digikey part number"

Commit message: Switched location of low side switches
Parts:
- added J11: Switch_D_High, footprints:Square_Pad_6mm, symbol Connector_Generic:Conn_01x01
- added J7: Switch_A_High, footprints:Square_Pad_6mm, symbol Connector_Generic:Conn_01x01
- added J8: Switch_B_High, footprints:Square_Pad_6mm, symbol Connector_Generic:Conn_01x01
- added J9: Switch_C_High, footprints:Square_Pad_6mm, symbol Connector_Generic:Conn_01x01
Connections:
- net labels added: SWITCH_A_HIGH, SWITCH_B_HIGH, SWITCH_C_HIGH, SWITCH_D_HIGH
- wire segments 309 -> 333

Commit message: added diode marks to diodes
Parts:
- D1, D2, D3, D4, D5, D6, D7, D8: footprint LED_SMD:LED_0603_1608Metric_Pad1.05x0.95mm_HandSolder -> footprints:LED_0603_1608Metric_Pad1.05x0.95mm_HandSolder_diode_mark
Changed lines of the file:
@@
 F 0 "D1" H 1792 5745 50  0000 C CNN
 F 1 "LED" H 1792 5836 50  0000 C CNN
-F 2 "LED_SMD:LED_0603_1608Metric_Pad1.05x0.95mm_HandSolder" H 1800 6000 50  0001 C CNN
+F 2 "footprints:LED_0603_1608Metric_Pad1.05x0.95mm_HandSolder_diode_mark" H 1800 6000 50  0001 C CNN
 F 3 "~" H 1800 6000 50  0001 C CNN
 	1    1800 6000
@@
 F 0 "D2" H 1792 6045 50  0000 C CNN
 F 1 "LED" H 1792 6136 50  0000 C CNN
-F 2 "LED_SMD:LED_0603_1608Metric_Pad1.05x0.95mm_HandSolder" H 1800 6300 50  0001 C CNN
+F 2 "footprints:LED_0603_1608Metric_Pad1.05x0.95mm_HandSolder_diode_mark" H 1800 6300 50  0001 C CNN
 F 3 "~" H 1800 6300 50  0001 C CNN
 	1    1800 6300
@@
 F 0 "D3" H 1792 6445 50  0000 C CNN
 F 1 "LED" H 1792 6536 50  0000 C CNN
-F 2 "LED_SMD:LED_0603_1608Metric_Pad1.05x0.95mm_HandSolder" H 1800 6700 50  0001 C CNN
+F 2 "footprints:LED_0603_1608Metric_Pad1.05x0.95mm_HandSolder_diode_mark" H 1800 6700 50  0001 C CNN
 F 3 "~" H 1800 6700 50  0001 C CNN
 	1    1800 6700
@@
 F 0 "D4" H 7242 8795 50  0000 C CNN
 F 1 "LED" H 7242 8886 50  0000 C CNN
-F 2 "LED_SMD:LED_0603_1608Metric_Pad1.05x0.95mm_HandSolder" H 7250 9050 50  0001 C CNN
+F 2 "footprints:LED_0603_1608Metric_Pad1.05x0.95mm_HandSolder_diode_mark" H 7250 9050 50  0001 C CNN
 F 3 "~" H 7250 9050 50  0001 C CNN
 	1    7250 9050
@@
 F 0 "D5" H 7242 9145 50  0000 C CNN
 F 1 "LED" H 7242 9236 50  0000 C CNN
-F 2 "LED_SMD:LED_0603_1608Metric_Pad1.05x0.95mm_HandSolder" H 7250 9400 50  0001 C CNN
+F 2 "footprints:LED_0603_1608Metric_Pad1.05x0.95mm_HandSolder_diode_mark" H 7250 9400 50  0001 C CNN
 F 3 "~" H 7250 9400 50  0001 C CNN
 	1    7250 9400
@@
 F 0 "D6" H 7242 9495 50  0000 C CNN
 F 1 "LED" H 7242 9586 50  0000 C CNN
-F 2 "LED_SMD:LED_0603_1608Metric_Pad1.05x0.95mm_HandSolder" H 7250 9750 50  0001 C CNN
+F 2 "footprints:LED_0603_1608Metric_Pad1.05x0.95mm_HandSolder_diode_mark" H 7250 9750 50  0001 C CNN
 F 3 "~" H 7250 9750 50  0001 C CNN
 	1    7250 9750
@@
 F 0 "D7" H 7242 9845 50  0000 C CNN
 F 1 "LED" H 7242 9936 50  0000 C CNN
-F 2 "LED_SMD:LED_0603_1608Metric_Pad1.05x0.95mm_HandSolder" H 7250 10100 50  0001 C CNN
+F 2 "footprints:LED_0603_1608Metric_Pad1.05x0.95mm_HandSolder_diode_mark" H 7250 10100 50  0001 C CNN
 F 3 "~" H 7250 10100 50  0001 C CNN
 	1    7250 10100
@@
 F 0 "D8" H 1792 6795 50  0000 C CNN
 F 1 "LED" H 1792 6886 50  0000 C CNN
-F 2 "LED_SMD:LED_0603_1608Metric_Pad1.05x0.95mm_HandSolder" H 1800 7050 50  0001 C CNN
+F 2 "footprints:LED_0603_1608Metric_Pad1.05x0.95mm_HandSolder_diode_mark" H 1800 7050 50  0001 C CNN
 F 3 "~" H 1800 7050 50  0001 C CNN
 	1    1800 7050
