File: electrical/control board power/_saved_control board power.sch (KiCad schematic (older format))
At the start: 67 parts, among them J1 Conn_01x02, J10 48V_from_conversion, J11 Aux_2, J17 Switch_B, J2 5V, J3 Barrel_Jack, J4 Switch_A, J5 Switch_Input, J6 Power_Connector, J7 Switch_A_High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

Commit message: odroid footprint now has correct pad dimentions
Parts:
- gave numbers to parts that had none: 1
Changed lines of the file:
@@
 Connection ~ 9400 8750
 $Comp
-L Connector_Generic:Conn_02x08_Odd_Even J?
+L Connector_Generic:Conn_02x08_Odd_Even J12
 U 1 1 5C7F656B
 P 9750 8950
-F 0 "J?" H 9800 9467 50  0000 C CNN
+F 0 "J12" H 9800 9467 50  0000 C CNN
 F 1 "Conn_02x08_Odd_Even" H 9800 9376 50  0000 C CNN
 F 2 "Connector_Harwin:Harwin_LTek-Male_2x08_P2.00mm_Vertical" H 9750 8950 50  0001 C CNN
